File: board2_monitor/board2_monitor.kicad_sch (KiCad schematic)
At the start: 0 parts

Commit message: board2_monitor: gauge matrix + IS31FL3731 driver + CA net-class colors (WIP)
- 72-LED charlieplex matrix wired across CA1-CA9 (Matrix A), all valid.
- IS31FL3731 (U1) gauge driver: VCC<-CH1_V, GND, SDA/SCL, AD->GND (0x74),
  IN->GND, CA1-CA9 -> matrix; CB1-CB9/INTB no-connected (Matrix B unused).
- Added 9 net-class colors for CA1-CA9 (readable palette) + patterns.
- Connectors J1s (SDA/SCL/WAKE/SGND) and power connectors in place.

WIP: SDB pull-up (R1 10k) and R_EXT (R2 20k) free ends still need to land on
U1 pins 3/6; a few dangling wires + PWR_FLAGs to clean.

Co-Authored-By: Claude Opus 4.8 (1M context) <noreply@anthropic.com>
Parts:
- added C1: 1uF, Capacitor_SMD:C_0603_1608Metric, symbol Device:C
- added C2: 0.1uf, Capacitor_SMD:C_0805_2012Metric, symbol Device:C
- added C3: 1uf, Capacitor_SMD:C_0805_2012Metric, symbol Device:C
- added D1, D10, D11, D12, D13, D14, D15, D16, D17, D18, D19, D2, D20, D21, D22, D23, D24, D25, D26, D27, D28, D29, D3, D30, D31, D32, D33, D34, D35, D36, D37, D38, D39, D4, D40, D41, D42, D43, D44, D45, D46, D47, D48, D49, D5, D50, D51, D52, D53, D54, D55, D56, D57, D58, D59, D6, D60, D61, D62, D63, D64, D65, D66, D67, D68, D69, D7, D70, D71, D72, D8, D9: LED, PCM_SparkFun-LED:LED_0603_1608Metric, symbol PCM_SparkFun-LED:LED
- added J1: Screw_Terminal_01x08, TerminalBlock_Phoenix:TerminalBlock_Phoenix_PT-1,5-8-3.5-H_1x08_P3.50mm_Horizontal, symbol Connector:Screw_Terminal_01x08
- added J2: Conn_01x04, Connector_PinSocket_2.54mm:PinSocket_1x04_P2.54mm_Vertical, symbol Connector_Generic:Conn_01x04
- added J3, J4: Conn_02x04_Odd_Even, Connector_PinSocket_2.54mm:PinSocket_2x04_P2.54mm_Vertical, symbol Connector_Generic:Conn_02x04_Odd_Even
- added R1: 10K, Resistor_SMD:R_0603_1608Metric, symbol Device:R
- added R2: 20K, Resistor_SMD:R_0603_1608Metric, symbol Device:R
- added SW1: WAKE, Button_Switch_SMD:SW_Push_1P1T_NO_CK_KMR2, symbol Switch:SW_Push
- added U1: IS31FL3731-SA, Package_SO:SSOP-28_5.3x10.2mm_P0.65mm, symbol Driver_LED:IS31FL3731-SA
Connections:
- new net: R2.1, U1.6 (R_EXT)
- new net: R1.1, U1.3 (~{SDB})
- new net: C1.1, U1.16 (C_FILT)
- new net CA1: D1.1 (K), D10.1 (K), D11.2 (A), D19.1 (K), D2.2 (A), D20.2 (A), D28.1 (K), D29.2 (A), D37.1 (K), D38.2 (A), D46.1 (K), D47.2 (A), D55.1 (K), D56.2 (A), D64.1 (K), D65.2 (A), U1.21 (CA1)
- new net CA2: D12.2 (A), D21.2 (A), D3.2 (A), D30.2 (A), D39.2 (A), D48.2 (A), D57.2 (A), D64.2 (A), D65.1 (K), D66.1 (K), D67.1 (K), D68.1 (K), D69.1 (K), D70.1 (K), D71.1 (K), D72.1 (K), U1.22 (CA2)
- new net CA3: D13.2 (A), D22.2 (A), D31.2 (A), D4.2 (A), D40.2 (A), D49.2 (A), D55.2 (A), D56.1 (K), D57.1 (K), D58.1 (K), D59.1 (K), D60.1 (K), D61.1 (K), D62.1 (K), D63.1 (K), D66.2 (A), U1.23 (CA3)
- new net CA4: D14.2 (A), D23.2 (A), D32.2 (A), D41.2 (A), D46.2 (A), D47.1 (K), D48.1 (K), D49.1 (K), D5.2 (A), D50.1 (K), D51.1 (K), D52.1 (K), D53.1 (K), D54.1 (K), D58.2 (A), D67.2 (A), U1.24 (CA4)
- new net CA5: D15.2 (A), D24.2 (A), D33.2 (A), D37.2 (A), D38.1 (K), D39.1 (K), D40.1 (K), D41.1 (K), D42.1 (K), D43.1 (K), D44.1 (K), D45.1 (K), D50.2 (A), D59.2 (A), D6.2 (A), D68.2 (A), U1.25 (CA5)
- new net CA6: D16.2 (A), D25.2 (A), D28.2 (A), D29.1 (K), D30.1 (K), D31.1 (K), D32.1 (K), D33.1 (K), D34.1 (K), D35.1 (K), D36.1 (K), D42.2 (A), D51.2 (A), D60.2 (A), D69.2 (A), D7.2 (A), U1.26 (CA6)
- new net CA7: D17.2 (A), D19.2 (A), D20.1 (K), D21.1 (K), D22.1 (K), D23.1 (K), D24.1 (K), D25.1 (K), D26.1 (K), D27.1 (K), D34.2 (A), D43.2 (A), D52.2 (A), D61.2 (A), D70.2 (A), D8.2 (A), U1.27 (CA7)
- new net CA8: D10.2 (A), D11.1 (K), D12.1 (K), D13.1 (K), D14.1 (K), D15.1 (K), D16.1 (K), D17.1 (K), D18.1 (K), D26.2 (A), D35.2 (A), D44.2 (A), D53.2 (A), D62.2 (A), D71.2 (A), D9.2 (A), U1.28 (CA8)
- new net CA9: D1.2 (A), D18.2 (A), D2.1 (K), D27.2 (A), D3.1 (K), D36.2 (A), D4.1 (K), D45.2 (A), D5.1 (K), D54.2 (A), D6.1 (K), D63.2 (A), D7.1 (K), D72.2 (A), D8.1 (K), D9.1 (K), U1.1 (CA9)
- new net CH1_V: C2.1, C3.1, J3.1 (Pin_1), R1.2, U1.2 (VCC)
- new net CH1_VIN: J1.1 (Pin_1), SW1.2
- new net CH1_VOUT: J1.2 (Pin_2), J4.1 (Pin_1)
- new net CH2_V: J1.3 (Pin_3), J3.3 (Pin_3)
- new net CH2_VOUT: J1.4 (Pin_4), J4.3 (Pin_3)
- new net CH3_V: J1.5 (Pin_5), J3.5 (Pin_5)
- new net CH3_VOUT: J1.6 (Pin_6), J4.5 (Pin_5)
- new net CH4_V: J1.7 (Pin_7), J3.7 (Pin_7)
- new net CH4_VOUT: J1.8 (Pin_8), J4.7 (Pin_7)
- new net GND: C1.2, C2.2, C3.2, J2.4 (Pin_4), J3.2 (Pin_2), J3.4 (Pin_4), J3.6 (Pin_6), J3.8 (Pin_8), J4.2 (Pin_2), J4.4 (Pin_4), J4.6 (Pin_6), J4.8 (Pin_8), R2.2, U1.17 (IN), U1.18 (AD), U1.5 (GND)
- new net SCL: J2.2 (Pin_2), U1.20 (SCL)
- new net SDA: J2.1 (Pin_1), U1.19 (SDA)
- new net WAKE: J2.3 (Pin_3), SW1.1
- no-connect marks 0 -> 10
Other:
- note added: "8X9 CHARLIEPLEXED LED MATRIX"
- note added: "ACTIVATE"
- note added: "BAT 1"
- note added: "BAT 2"
- note added: "BAT 3"
- note added: "BAT 4"
- note added: "DATA"
- note added: "DUAL 8X9 CHARLIEPLEXED LED MATRIX DRIVER"
- note added: "LED DRIVER"
- note added: "LED MATRIX"
- note added: "POWER IN"
- note added: "POWER OUT"
- note added: "PULL PINS"

Commit message: board2_monitor: gauge matrix layout + LED designators corrected (column-major, 9 per column)
Co-Authored-By: Claude Opus 4.8 (1M context) <noreply@anthropic.com>
Parts:
- C1: footprint Capacitor_SMD:C_0603_1608Metric -> Capacitor_SMD:C_0805_2012Metric
- R1, R2: footprint Resistor_SMD:R_0603_1608Metric -> Resistor_SMD:R_0805_2012Metric
- renumbered C3 to C2, C2 to C3, J3 to J1, J4 to J2, J2 to J3, J1 to J4
Connections:
- net CH1_VIN is gone; now on net CH1_V: J4.1 (Pin_1), SW1.2
- net CA1: now also D1.2 (A), D18.2 (A), D2.1 (K), D27.2 (A), D3.1 (K), D36.2 (A), D4.1 (K), D45.2 (A), D5.1 (K), D54.2 (A), D6.1 (K), D63.2 (A), D7.1 (K), D72.2 (A), D8.1 (K), D9.1 (K); no longer D1.1 (K), D10.1 (K), D11.2 (A), D19.1 (K), D2.2 (A), D20.2 (A), D28.1 (K), D29.2 (A), D37.1 (K), D38.2 (A), D46.1 (K), D47.2 (A), D55.1 (K), D56.2 (A), D64.1 (K), D65.2 (A)
- net CA2: now also D10.2 (A), D11.1 (K), D12.1 (K), D13.1 (K), D14.1 (K), D15.1 (K), D16.1 (K), D17.1 (K), D18.1 (K), D26.2 (A), D35.2 (A), D44.2 (A), D53.2 (A), D62.2 (A), D71.2 (A), D9.2 (A); no longer D12.2 (A), D21.2 (A), D3.2 (A), D30.2 (A), D39.2 (A), D48.2 (A), D57.2 (A), D64.2 (A), D65.1 (K), D66.1 (K), D67.1 (K), D68.1 (K), D69.1 (K), D70.1 (K), D71.1 (K), D72.1 (K)
- net CA3: now also D17.2 (A), D19.2 (A), D20.1 (K), D21.1 (K), D22.1 (K), D23.1 (K), D24.1 (K), D25.1 (K), D26.1 (K), D27.1 (K), D34.2 (A), D43.2 (A), D52.2 (A), D61.2 (A), D70.2 (A), D8.2 (A); no longer D13.2 (A), D22.2 (A), D31.2 (A), D4.2 (A), D40.2 (A), D49.2 (A), D55.2 (A), D56.1 (K), D57.1 (K), D58.1 (K), D59.1 (K), D60.1 (K), D61.1 (K), D62.1 (K), D63.1 (K), D66.2 (A)
- net CA4: now also D16.2 (A), D25.2 (A), D28.2 (A), D29.1 (K), D30.1 (K), D31.1 (K), D32.1 (K), D33.1 (K), D34.1 (K), D35.1 (K), D36.1 (K), D42.2 (A), D51.2 (A), D60.2 (A), D69.2 (A), D7.2 (A); no longer D14.2 (A), D23.2 (A), D32.2 (A), D41.2 (A), D46.2 (A), D47.1 (K), D48.1 (K), D49.1 (K), D5.2 (A), D50.1 (K), D51.1 (K), D52.1 (K), D53.1 (K), D54.1 (K), D58.2 (A), D67.2 (A)
- net CA6: now also D14.2 (A), D23.2 (A), D32.2 (A), D41.2 (A), D46.2 (A), D47.1 (K), D48.1 (K), D49.1 (K), D5.2 (A), D50.1 (K), D51.1 (K), D52.1 (K), D53.1 (K), D54.1 (K), D58.2 (A), D67.2 (A); no longer D16.2 (A), D25.2 (A), D28.2 (A), D29.1 (K), D30.1 (K), D31.1 (K), D32.1 (K), D33.1 (K), D34.1 (K), D35.1 (K), D36.1 (K), D42.2 (A), D51.2 (A), D60.2 (A), D69.2 (A), D7.2 (A)
- net CA7: now also D13.2 (A), D22.2 (A), D31.2 (A), D4.2 (A), D40.2 (A), D49.2 (A), D55.2 (A), D56.1 (K), D57.1 (K), D58.1 (K), D59.1 (K), D60.1 (K), D61.1 (K), D62.1 (K), D63.1 (K), D66.2 (A); no longer D17.2 (A), D19.2 (A), D20.1 (K), D21.1 (K), D22.1 (K), D23.1 (K), D24.1 (K), D25.1 (K), D26.1 (K), D27.1 (K), D34.2 (A), D43.2 (A), D52.2 (A), D61.2 (A), D70.2 (A), D8.2 (A)
- net CA8: now also D12.2 (A), D21.2 (A), D3.2 (A), D30.2 (A), D39.2 (A), D48.2 (A), D57.2 (A), D64.2 (A), D65.1 (K), D66.1 (K), D67.1 (K), D68.1 (K), D69.1 (K), D70.1 (K), D71.1 (K), D72.1 (K); no longer D10.2 (A), D11.1 (K), D12.1 (K), D13.1 (K), D14.1 (K), D15.1 (K), D16.1 (K), D17.1 (K), D18.1 (K), D26.2 (A), D35.2 (A), D44.2 (A), D53.2 (A), D62.2 (A), D71.2 (A), D9.2 (A)
- net CA9: now also D1.1 (K), D10.1 (K), D11.2 (A), D19.1 (K), D2.2 (A), D20.2 (A), D28.1 (K), D29.2 (A), D37.1 (K), D38.2 (A), D46.1 (K), D47.2 (A), D55.1 (K), D56.2 (A), D64.1 (K), D65.2 (A); no longer D1.2 (A), D18.2 (A), D2.1 (K), D27.2 (A), D3.1 (K), D36.2 (A), D4.1 (K), D45.2 (A), D5.1 (K), D54.2 (A), D6.1 (K), D63.2 (A), D7.1 (K), D72.2 (A), D8.1 (K), D9.1 (K)
- net CH1_V: now also J1.7 (Pin_7); no longer J1.1 (Pin_1)
- net CH1_VOUT: now also J2.7 (Pin_7); no longer J2.1 (Pin_1)
- net CH2_V: now also J1.5 (Pin_5); no longer J1.3 (Pin_3)
- net CH2_VOUT: now also J2.5 (Pin_5); no longer J2.3 (Pin_3)
- net CH3_V: now also J1.3 (Pin_3); no longer J1.5 (Pin_5)
- net CH3_VOUT: now also J2.3 (Pin_3); no longer J2.5 (Pin_5)
- net CH4_V: now also J1.1 (Pin_1); no longer J1.7 (Pin_7)
- net CH4_VOUT: now also J2.1 (Pin_1); no longer J2.7 (Pin_7)
Changed lines of the file:
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@@
 	)
 	(label "CA2"
-		(at 111.125 60.96 0)
+		(at 111.125 111.76 0)
 		(effects
 			(font
@@
 	)
 	(label "CH2_V"
-		(at 31.115 146.685 0)
+		(at 31.115 149.225 0)
 		(effects
 			(font
@@
 		)
 	)
-	(label "CH1_VIN"
+	(label "CH1_V"
 		(at 241.3 147.955 180)
 		(effects
@@
 	)
 	(label "CA7"
-		(at 111.125 99.06 0)
+		(at 111.125 68.58 0)
 		(effects
 			(font
@@
 	)
 	(label "CH3_V"
-		(at 31.115 149.225 0)
+		(at 31.115 146.685 0)
 		(effects
 			(font
@@
 	)
 	(label "CH1_VOUT"
-		(at 76.835 144.145 0)
+		(at 76.835 151.765 0)
 		(effects
 			(font
@@
 	)
 	(label "CA9"
-		(at 111.125 119.38 0)
+		(at 111.125 53.34 0)
 		(effects
 			(font
@@
 	)
 	(label "CH4_V"
-		(at 31.115 151.765 0)
+		(at 31.115 144.145 0)
 		(effects
 			(font
@@
 	)
 	(label "CH1_V"
-		(at 31.115 144.145 0)
+		(at 31.115 151.765 0)
 		(effects
 			(font
@@
 	)
 	(label "CH2_VOUT"
-		(at 76.835 146.685 0)
+		(at 76.835 149.225 0)
 		(effects
 			(font
@@
 	)
 	(label "CA8"
-		(at 111.125 111.76 0)
+		(at 111.125 60.96 0)
 		(effects
 			(font
@@
 	)
 	(label "CA1"
-		(at 111.125 53.34 0)
+		(at 111.125 119.38 0)
 		(effects
 			(font
@@
 	)
 	(label "CH4_VOUT"
-		(at 76.835 151.765 0)
+		(at 76.835 144.145 0)
 		(effects
 			(font
@@
 	)
 	(label "CH3_VOUT"
-		(at 76.835 149.225 0)
+		(at 76.835 146.685 0)
 		(effects
 			(font
@@
 	)
 	(label "CA6"
-		(at 111.125 91.44 0)
+		(at 111.125 76.2 0)
 		(effects
 			(font
@@
 		)
 	)
-	(label "CH1_VIN"
+	(label "CH1_V"
 		(at 173.99 139.065 0)
 		(effects
@@
 	)
 	(label "CA3"
-		(at 111.125 68.58 0)
+		(at 111.125 99.06 0)
 		(effects
 			(font
@@
 	)
 	(label "CA4"
-		(at 111.125 76.2 0)
+		(at 111.125 91.44 0)
 		(effects
 			(font
@@
 		)
 	)
+	(rule_area
+		(exclude_from_sim no)
+		(in_bom yes)
+		(on_board yes)
+		(dnp no)
+		(polyline
+			(pts
+				(xy 146.685 37.465) (xy 146.685 114.935) (xy 120.65 114.935) (xy 120.65 37.465)
+			)
+			(stroke
+				(width 0)
+				(type dash)
+			)
+			(fill
+				(type none)
+			)
+		)
+	)
 	(symbol
 		(lib_id "PCM_SparkFun-LED:LED")
@@
 		(dnp no)
 		(fields_autoplaced yes)
-		(property "Reference" "#PWR013"
+		(property "Reference" "#PWR01"
 			(at 30.48 73.66 0)
 			(hide yes)
@@
 			(project "board2_monitor"
 				(path "/0d1390b9-e848-4ad4-8bef-84851d0f73a3"
-					(reference "#PWR013")
+					(reference "#PWR01")
 					(unit 1)
 				)
@@
 			)
 		)
-		(property "Footprint" "Resistor_SMD:R_0603_1608Metric"
+		(property "Footprint" "Resistor_SMD:R_0805_2012Metric"
 			(at 43.18 79.502 90)
 			(hide yes)
@@
 		(dnp no)
 		(fields_autoplaced yes)
-		(property "Reference" "#PWR02"
+		(property "Reference" "#PWR07"
 			(at 63.5 146.685 0)
 			(hide yes)
@@
 			(project "board2_monitor"
 				(path "/0d1390b9-e848-4ad4-8bef-84851d0f73a3"
-					(reference "#PWR02")
+					(reference "#PWR07")
 					(unit 1)
 				)
@@
 		(dnp no)
 		(fields_autoplaced yes)
-		(property "Reference" "#PWR011"
+		(property "Reference" "#PWR05"
 			(at 43.18 60.96 0)
 			(hide yes)
@@
 			(project "board2_monitor"
 				(path "/0d1390b9-e848-4ad4-8bef-84851d0f73a3"
-					(reference "#PWR011")
+					(reference "#PWR05")
 					(unit 1)
 				)
@@
 		(dnp no)
 		(fields_autoplaced yes)
-		(property "Reference" "C2"
+		(property "Reference" "C3"
 			(at 54.61 42.5449 0)
 			(show_name no)
@@
 			(project "board2_monitor"
 				(path "/0d1390b9-e848-4ad4-8bef-84851d0f73a3"
-					(reference "C2")
+					(reference "C3")
 					(unit 1)
 				)
@@
 		(in_pos_files yes)
 		(dnp no)
-		(property "Reference" "C3"
+		(property "Reference" "C2"
 			(at 41.91 42.5449 0)
 			(show_name no)
@@
 			(project "board2_monitor"
 				(path "/0d1390b9-e848-4ad4-8bef-84851d0f73a3"
-					(reference "C3")
+					(reference "C2")
 					(unit 1)
 				)
@@
 		(dnp no)
 		(fields_autoplaced yes)
-		(property "Reference" "#PWR03"
+		(property "Reference" "#PWR08"
 			(at 63.5 149.225 0)
 			(hide yes)
@@
 			(project "board2_monitor"
 				(path "/0d1390b9-e848-4ad4-8bef-84851d0f73a3"
-					(reference "#PWR03")
+					(reference "#PWR08")
 					(unit 1)
 				)
@@
 		(in_pos_files yes)
 		(dnp no)
-		(property "Reference" "J1"
+		(property "Reference" "J4"
 			(at 192.405 146.6849 0)
 			(show_name no)
@@
 			(project "board2_monitor"
 				(path "/0d1390b9-e848-4ad4-8bef-84851d0f73a3"
-					(reference "J1")
+					(reference "J4")
 					(unit 1)
 				)
@@
 		(dnp no)
 		(fields_autoplaced yes)
-		(property "Reference" "#PWR06"
+		(property "Reference" "#PWR011"
 			(at 109.22 144.145 0)
 			(hide yes)
@@
 			(project "board2_monitor"
 				(path "/0d1390b9-e848-4ad4-8bef-84851d0f73a3"
-					(reference "#PWR06")
+					(reference "#PWR011")
 					(unit 1)
 				)
@@
 		(dnp no)
 		(fields_autoplaced yes)
-		(property "Reference" "#PWR04"
+		(property "Reference" "#PWR09"
 			(at 63.5 151.765 0)
 			(hide yes)
@@
 			(project "board2_monitor"
 				(path "/0d1390b9-e848-4ad4-8bef-84851d0f73a3"
-					(reference "#PWR04")
+					(reference "#PWR09")
 					(unit 1)
 				)
@@
 			)
 		)
-		(property "Footprint" "Resistor_SMD:R_0603_1608Metric"
+		(property "Footprint" "Resistor_SMD:R_0805_2012Metric"
 			(at 43.18 64.262 90)
 			(hide yes)
@@
 		(dnp no)
 		(fields_autoplaced yes)
-		(property "Reference" "#PWR01"
+		(property "Reference" "#PWR06"
 			(at 63.5 144.145 0)
 			(hide yes)
@@
 			(project "board2_monitor"
 				(path "/0d1390b9-e848-4ad4-8bef-84851d0f73a3"
-					(reference "#PWR01")
+					(reference "#PWR06")
 					(unit 1)
 				)
@@
 		(dnp no)
 		(fields_autoplaced yes)
-		(property "Reference" "#PWR08"
+		(property "Reference" "#PWR013"
 			(at 109.22 149.225 0)
 			(hide yes)
@@
 			(project "board2_monitor"
 				(path "/0d1390b9-e848-4ad4-8bef-84851d0f73a3"
-					(reference "#PWR08")
+					(reference "#PWR013")
 					(unit 1)
 				)
@@
 		(in_pos_files yes)
 		(dnp no)
-		(property "Reference" "J4"
+		(property "Reference" "J2"
 			(at 93.345 137.795 0)
 			(show_name no)
@@
 			(project "board2_monitor"
 				(path "/0d1390b9-e848-4ad4-8bef-84851d0f73a3"
-					(reference "J4")
+					(reference "J2")
 					(unit 1)
 				)
@@
 		(dnp no)
 		(fields_autoplaced yes)
-		(property "Reference" "#PWR05"
+		(property "Reference" "#PWR015"
 			(at 130.175 149.86 0)
 			(hide yes)
@@
 			(project "board2_monitor"
 				(path "/0d1390b9-e848-4ad4-8bef-84851d0f73a3"
-					(reference "#PWR05")
+					(reference "#PWR015")
 					(unit 1)
 				)
@@
 		(dnp no)
 		(fields_autoplaced yes)
-		(property "Reference" "#PWR015"
+		(property "Reference" "#PWR04"
 			(at 48.26 29.845 0)
 			(hide yes)
@@
 			(project "board2_monitor"
 				(path "/0d1390b9-e848-4ad4-8bef-84851d0f73a3"
-					(reference "#PWR015")
+					(reference "#PWR04")
 					(unit 1)
 				)
@@
 		(dnp no)
 		(fields_autoplaced yes)
-		(property "Reference" "#PWR09"
+		(property "Reference" "#PWR014"
 			(at 109.22 151.765 0)
 			(hide yes)
@@
 			(project "board2_monitor"
 				(path "/0d1390b9-e848-4ad4-8bef-84851d0f73a3"
-					(reference "#PWR09")
+					(reference "#PWR014")
 					(unit 1)
 				)
@@
 		(dnp no)
 		(fields_autoplaced yes)
-		(property "Reference" "#PWR012"
+		(property "Reference" "#PWR03"
 			(at 30.48 81.28 0)
 			(hide yes)
@@
 			(project "board2_monitor"
 				(path "/0d1390b9-e848-4ad4-8bef-84851d0f73a3"
-					(reference "#PWR012")
+					(reference "#PWR03")
 					(unit 1)
 				)
@@
 		(dnp no)
 		(fields_autoplaced yes)
-		(property "Reference" "#PWR07"
+		(property "Reference" "#PWR012"
 			(at 109.22 146.685 0)
 			(hide yes)
@@
 			(project "board2_monitor"
 				(path "/0d1390b9-e848-4ad4-8bef-84851d0f73a3"
-					(reference "#PWR07")
+					(reference "#PWR012")
 					(unit 1)
 				)
@@
 			)
 		)
-		(property "Footprint" "Capacitor_SMD:C_0603_1608Metric"
+		(property "Footprint" "Capacitor_SMD:C_0805_2012Metric"
 			(at 39.37 77.1652 0)
 			(hide yes)
@@
 		(dnp no)
 		(fields_autoplaced yes)
-		(property "Reference" "#PWR014"
+		(property "Reference" "#PWR02"
 			(at 30.48 76.2 0)
 			(hide yes)
@@
 			(project "board2_monitor"
 				(path "/0d1390b9-e848-4ad4-8bef-84851d0f73a3"
-					(reference "#PWR014")
+					(reference "#PWR02")
 					(unit 1)
 				)
@@
 		(dnp no)
 		(fields_autoplaced yes)
-		(property "Reference" "J2"
+		(property "Reference" "J3"
 			(at 144.78 144.7799 0)
 			(show_name no)
@@
 			(project "board2_monitor"
 				(path "/0d1390b9-e848-4ad4-8bef-84851d0f73a3"
-					(reference "J2")
+					(reference "J3")
 					(unit 1)
 				)
@@
 		(dnp no)
 		(fields_autoplaced yes)
-		(property "Reference" "J3"
+		(property "Reference" "J1"
 			(at 47.625 137.795 0)
 			(show_name no)
@@
 			(project "board2_monitor"
 				(path "/0d1390b9-e848-4ad4-8bef-84851d0f73a3"
-					(reference "J3")
+					(reference "J1")
 					(unit 1)
 				)
@@
 		)
 	)
+	(group ""
+		(members "024d17b1-126e-4630-acb8-9e3124bb105b" "13ce72be-8471-41b1-90ac-7cad2a7f6772"
+			"19edd71f-0d75-4565-8ce6-29b74b022ca7" "1edb52f9-e41e-4d8b-8005-b9bbc50f976d"
+			"27642fc3-b222-4ae0-b03c-78928e4c55ff" "2933783a-d457-4f48-ab48-162180164315"
+			"37437ef5-3f27-4d26-bde6-7564dd5b51ba" "3caf3d99-f337-4120-b809-945f507b86c7"
+			"623be199-adda-4087-b77a-3e966c172eee" "a2779ec4-9ecf-4485-ba64-a987e2ab313f"
+			"aebc1b33-c8ca-468e-b471-2ae67f13f393" "b9028484-abca-439d-b575-b268aa9351f4"
+			"c6da93df-865e-45ac-b250-bafecd0cdce7" "c7937c40-c334-4c2c-9e34-47739af39191"
+			"c9ff51cf-ed88-40a8-9dde-69fad38569d9" "d251f6b1-7fc4-4603-bc10-fe6e0ed60ef3"
+			"da2c96a9-8370-47e5-87f7-d52213ce98a9" "f6ecbc79-67a0-419e-a3cd-553228bd66eb"
+			"fe7e9fe6-e89f-499c-af16-0a5a52864a59"
+		)
+	)
