File: board2_monitor/board2_monitor.kicad_pcb (KiCad board)
At the start: 0 parts

Commit message: board2_monitor: gauge matrix layout + LED designators corrected (column-major, 9 per column)
Co-Authored-By: Claude Opus 4.8 (1M context) <noreply@anthropic.com>
Parts:
- added C1: 1uF, Capacitor_SMD:C_0805_2012Metric, F.Cu at (126.5, 71.3)
- added C2: 1uf, Capacitor_SMD:C_0805_2012Metric, F.Cu at (132.1, 58.6)
- added C3: 0.1uf, Capacitor_SMD:C_0805_2012Metric, F.Cu at (134.1, 58.6)
- added D1: LED, PCM_SparkFun-LED:LED_0603_1608Metric, F.Cu at (115.8, 75.3)
- added D10: LED, PCM_SparkFun-LED:LED_0603_1608Metric, F.Cu at (120.0, 75.3)
- added D11: LED, PCM_SparkFun-LED:LED_0603_1608Metric, F.Cu at (120.0, 76.9)
- added D12: LED, PCM_SparkFun-LED:LED_0603_1608Metric, F.Cu at (120.0, 78.4)
- added D13: LED, PCM_SparkFun-LED:LED_0603_1608Metric, F.Cu at (120.0, 80.0)
- added D14: LED, PCM_SparkFun-LED:LED_0603_1608Metric, F.Cu at (120.0, 81.5)
- added D15: LED, PCM_SparkFun-LED:LED_0603_1608Metric, F.Cu at (120.0, 83.0)
- added D16: LED, PCM_SparkFun-LED:LED_0603_1608Metric, F.Cu at (120.0, 84.6)
- added D17: LED, PCM_SparkFun-LED:LED_0603_1608Metric, F.Cu at (120.0, 86.2)
- added D18: LED, PCM_SparkFun-LED:LED_0603_1608Metric, F.Cu at (120.0, 88.8)
- added D19: LED, PCM_SparkFun-LED:LED_0603_1608Metric, F.Cu at (124.5, 75.3)
- added D2: LED, PCM_SparkFun-LED:LED_0603_1608Metric, F.Cu at (115.8, 76.9)
- added D20: LED, PCM_SparkFun-LED:LED_0603_1608Metric, F.Cu at (124.5, 76.9)
- added D21: LED, PCM_SparkFun-LED:LED_0603_1608Metric, F.Cu at (124.5, 78.4)
- added D22: LED, PCM_SparkFun-LED:LED_0603_1608Metric, F.Cu at (124.5, 80.0)
- added D23: LED, PCM_SparkFun-LED:LED_0603_1608Metric, F.Cu at (124.5, 81.5)
- added D24: LED, PCM_SparkFun-LED:LED_0603_1608Metric, F.Cu at (124.5, 83.0)
- added D25: LED, PCM_SparkFun-LED:LED_0603_1608Metric, F.Cu at (124.5, 84.6)
- added D26: LED, PCM_SparkFun-LED:LED_0603_1608Metric, F.Cu at (124.5, 86.2)
- added D27: LED, PCM_SparkFun-LED:LED_0603_1608Metric, F.Cu at (124.5, 88.8)
- added D28: LED, PCM_SparkFun-LED:LED_0603_1608Metric, F.Cu at (128.7, 75.3)
- added D29: LED, PCM_SparkFun-LED:LED_0603_1608Metric, F.Cu at (128.7, 76.9)
- added D3: LED, PCM_SparkFun-LED:LED_0603_1608Metric, F.Cu at (115.8, 78.4)
- added D30: LED, PCM_SparkFun-LED:LED_0603_1608Metric, F.Cu at (128.7, 78.4)
- added D31: LED, PCM_SparkFun-LED:LED_0603_1608Metric, F.Cu at (128.7, 80.0)
- added D32: LED, PCM_SparkFun-LED:LED_0603_1608Metric, F.Cu at (128.7, 81.5)
- added D33: LED, PCM_SparkFun-LED:LED_0603_1608Metric, F.Cu at (128.7, 83.0)
- added D34: LED, PCM_SparkFun-LED:LED_0603_1608Metric, F.Cu at (128.7, 84.6)
- added D35: LED, PCM_SparkFun-LED:LED_0603_1608Metric, F.Cu at (128.7, 86.2)
- added D36: LED, PCM_SparkFun-LED:LED_0603_1608Metric, F.Cu at (128.7, 88.8)
- added D37: LED, PCM_SparkFun-LED:LED_0603_1608Metric, F.Cu at (133.2, 75.3)
- added D38: LED, PCM_SparkFun-LED:LED_0603_1608Metric, F.Cu at (133.2, 76.9)
- added D39: LED, PCM_SparkFun-LED:LED_0603_1608Metric, F.Cu at (133.2, 78.4)
- added D4: LED, PCM_SparkFun-LED:LED_0603_1608Metric, F.Cu at (115.8, 80.0)
- added D40: LED, PCM_SparkFun-LED:LED_0603_1608Metric, F.Cu at (133.2, 80.0)
- added D41: LED, PCM_SparkFun-LED:LED_0603_1608Metric, F.Cu at (133.2, 81.5)
- added D42: LED, PCM_SparkFun-LED:LED_0603_1608Metric, F.Cu at (133.2, 83.0)
- added D43: LED, PCM_SparkFun-LED:LED_0603_1608Metric, F.Cu at (133.2, 84.6)
- added D44: LED, PCM_SparkFun-LED:LED_0603_1608Metric, F.Cu at (133.2, 86.2)
- added D45: LED, PCM_SparkFun-LED:LED_0603_1608Metric, F.Cu at (133.2, 88.8)
- added D46: LED, PCM_SparkFun-LED:LED_0603_1608Metric, F.Cu at (137.4, 75.3)
- added D47: LED, PCM_SparkFun-LED:LED_0603_1608Metric, F.Cu at (137.4, 76.9)
- added D48: LED, PCM_SparkFun-LED:LED_0603_1608Metric, F.Cu at (137.4, 78.4)
- added D49: LED, PCM_SparkFun-LED:LED_0603_1608Metric, F.Cu at (137.4, 80.0)
- added D5: LED, PCM_SparkFun-LED:LED_0603_1608Metric, F.Cu at (115.8, 81.5)
- added D50: LED, PCM_SparkFun-LED:LED_0603_1608Metric, F.Cu at (137.4, 81.5)
- added D51: LED, PCM_SparkFun-LED:LED_0603_1608Metric, F.Cu at (137.4, 83.0)
- added D52: LED, PCM_SparkFun-LED:LED_0603_1608Metric, F.Cu at (137.4, 84.6)
- added D53: LED, PCM_SparkFun-LED:LED_0603_1608Metric, F.Cu at (137.4, 86.2)
- added D54: LED, PCM_SparkFun-LED:LED_0603_1608Metric, F.Cu at (137.4, 88.8)
- added D55: LED, PCM_SparkFun-LED:LED_0603_1608Metric, F.Cu at (141.8, 75.3)
- added D56: LED, PCM_SparkFun-LED:LED_0603_1608Metric, F.Cu at (141.8, 76.9)
- added D57: LED, PCM_SparkFun-LED:LED_0603_1608Metric, F.Cu at (141.8, 78.4)
- added D58: LED, PCM_SparkFun-LED:LED_0603_1608Metric, F.Cu at (141.8, 80.0)
- added D59: LED, PCM_SparkFun-LED:LED_0603_1608Metric, F.Cu at (141.8, 81.5)
- added D6: LED, PCM_SparkFun-LED:LED_0603_1608Metric, F.Cu at (115.8, 83.0)
- added D60: LED, PCM_SparkFun-LED:LED_0603_1608Metric, F.Cu at (141.8, 83.0)
- added D61: LED, PCM_SparkFun-LED:LED_0603_1608Metric, F.Cu at (141.8, 84.6)
- added D62: LED, PCM_SparkFun-LED:LED_0603_1608Metric, F.Cu at (141.8, 86.2)
- added D63: LED, PCM_SparkFun-LED:LED_0603_1608Metric, F.Cu at (141.8, 88.8)
- added D64: LED, PCM_SparkFun-LED:LED_0603_1608Metric, F.Cu at (146.0, 75.3)
- added D65: LED, PCM_SparkFun-LED:LED_0603_1608Metric, F.Cu at (146.0, 76.9)
- added D66: LED, PCM_SparkFun-LED:LED_0603_1608Metric, F.Cu at (146.0, 78.4)
- added D67: LED, PCM_SparkFun-LED:LED_0603_1608Metric, F.Cu at (146.0, 80.0)
- added D68: LED, PCM_SparkFun-LED:LED_0603_1608Metric, F.Cu at (146.0, 81.5)
- added D69: LED, PCM_SparkFun-LED:LED_0603_1608Metric, F.Cu at (146.0, 83.0)
- added D7: LED, PCM_SparkFun-LED:LED_0603_1608Metric, F.Cu at (115.8, 84.6)
- added D70: LED, PCM_SparkFun-LED:LED_0603_1608Metric, F.Cu at (146.0, 84.6)
- added D71: LED, PCM_SparkFun-LED:LED_0603_1608Metric, F.Cu at (146.0, 86.2)
- added D72: LED, PCM_SparkFun-LED:LED_0603_1608Metric, F.Cu at (146.0, 88.8)
- added D8: LED, PCM_SparkFun-LED:LED_0603_1608Metric, F.Cu at (115.8, 86.2)
- added D9: LED, PCM_SparkFun-LED:LED_0603_1608Metric, F.Cu at (115.8, 88.8)
- added J1: Conn_02x04_Odd_Even, Connector_PinSocket_2.54mm:PinSocket_2x04_P2.54mm_Vertical, F.Cu at (132.8, 96.4)
- added J2: Conn_02x04_Odd_Even, Connector_PinSocket_2.54mm:PinSocket_2x04_P2.54mm_Vertical, F.Cu at (132.8, 118.0)
- added J3: Conn_01x04, Connector_PinSocket_2.54mm:PinSocket_1x04_P2.54mm_Vertical, F.Cu at (145.4, 96.4)
- added J4: Screw_Terminal_01x08, TerminalBlock_Phoenix:TerminalBlock_Phoenix_PT-1,5-8-3.5-H_1x08_P3.50mm_Horizontal, F.Cu at (144.3, 129.2)
- added R1: 10K, Resistor_SMD:R_0805_2012Metric, F.Cu at (130.1, 58.6)
- added R2: 20K, Resistor_SMD:R_0805_2012Metric, F.Cu at (128.1, 58.6)
- added SW1: WAKE, Button_Switch_SMD:SW_Push_1P1T_NO_CK_KMR2, F.Cu at (141.8, 65.5)
- added U1: IS31FL3731-SA, Package_SO:SSOP-28_5.3x10.2mm_P0.65mm, F.Cu at (129.6, 65.5)
Routing:
- net /CH1_V: track 0.00 -> 120.6 mm
- net /CA9: track 0.00 -> 89.7 mm, vias 0 -> 16
- net /CA8: track 0.00 -> 86.0 mm, vias 0 -> 16
- net /CA2: track 0.00 -> 81.7 mm, vias 0 -> 16
- net /CA7: track 0.00 -> 78.1 mm, vias 0 -> 16
- net /CA3: track 0.00 -> 77.6 mm, vias 0 -> 16
- net /CA6: track 0.00 -> 76.4 mm, vias 0 -> 16
- net /CA4: track 0.00 -> 75.2 mm, vias 0 -> 16
- net /CA5: track 0.00 -> 73.9 mm, vias 0 -> 16
- net /CA1: track 0.00 -> 64.6 mm, vias 0 -> 16
- net /WAKE: track 0.00 -> 46.6 mm
- net /SDA: track 0.00 -> 43.7 mm, vias 0 -> 1
- net /SCL: track 0.00 -> 39.0 mm, vias 0 -> 1
- net /CH2_V: track 0.00 -> 34.9 mm
- net /CH3_V: track 0.00 -> 25.8 mm
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- added copper zone on In1.Cu, net GND
Other:
- board outline added: 76 x 90 mm
- copper layers 0 -> 4
- board text added: "BATT 1"
- board text added: "BATT 1 +"
- board text added: "BATT 1 -"
- board text added: "BATT 2"
- board text added: "BATT 2 +"
- board text added: "BATT 2 -"
- board text added: "BATT 3"
- board text added: "BATT 3 +"
- board text added: "BATT 3 -"
- board text added: "BATT 4"
- board text added: "BATT 4 +"
- board text added: "BATT 4 -"
- board text added: "ERROR"
- board text added: "STATUS"
- board text added: "WAKE"

Commit message: board2_monitor: place UNSW Rocketry logo (small)
Co-Authored-By: Claude Opus 4.8 (1M context) <noreply@anthropic.com>
Parts:
- added G***: LOGO, UNSW_ROCKETRY_LIBRARY:ROCKETRY_LOGO_SMALL, F.Cu at (129.0, 105.9)
Other:
- board text added: "BY DASHIELL RUSSELL"
- board text added: "PULL PIN, DISTRUBUTION AND MONITORING BOARD"
- board text added: "UNSW AURC BMS"
Changed lines of the file:
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@@
 		)
 	)
+	(footprint "UNSW_ROCKETRY_LIBRARY:ROCKETRY_LOGO_SMALL"
+		(layer "F.Cu")
+		(at 129 105.9)
+		(property "Reference" "G***"
+			(at 0 0 0)
+			(layer "F.SilkS")
+			(hide yes)
+			(effects
+				(font
+					(size 1.5 1.5)
+					(thickness 0.3)
+				)
+			)
+		)
+		(property "Value" "LOGO"
+			(at 0.75 0 0)
+			(layer "F.SilkS")
+			(hide yes)
+			(effects
+				(font
+					(size 1.5 1.5)
+					(thickness 0.3)
+				)
+			)
+		)
+		(property "Datasheet" ""
+			(at 0 0 0)
+			(layer "F.Fab")
+			(hide yes)
+			(effects
+				(font
+					(size 1.27 1.27)
+				)
+			)
+		)
+		(property "Description" ""
+			(at 0 0 0)
+			(layer "F.Fab")
+			(hide yes)
+			(effects
+				(font
+					(size 1.27 1.27)
+				)
+			)
+		)
+		(attr board_only exclude_from_pos_files exclude_from_bom)
+		(duplicate_pad_numbers_are_jumpers no)
+		(fp_poly
+			(pts
+				(xy 1.558399 4.071777) (xy 1.81442 4.200328) (xy 2.039006 4.315338) (xy 2.219488 4.410131) (xy 2.343196 4.478036)
+				(xy 2.397462 4.512377) (xy 2.398878 4.514511) (xy 2.35736 4.537996) (xy 2.241866 4.590378) (xy 2.065976 4.666144)
+				(xy 1.843268 4.759783) (xy 1.587323 4.865782) (xy 1.311719 4.978629) (xy 1.030037 5.092812) (xy 0.755856 5.20282)
+				(xy 0.502756 5.303141) (xy 0.284315 5.388261) (xy 0.114114 5.45267) (xy 0.005732 5.490855) (xy -0.02655 5.499004)
+				(xy -0.0802 5.480681) (xy -0.209006 5.431236) (xy -0.401139 5.355376) (xy -0.644769 5.257809) (xy -0.928069 5.143242)
+				(xy -1.234722 5.018218) (xy -1.543115 4.891073) (xy -1.820828 4.774796) (xy -2.056561 4.674262)
+				(xy -2.239015 4.594347) (xy -2.356891 4.539927) (xy -2.398888 4.515878) (xy -2.398889 4.515854)
+				(xy -2.358775 4.487998) (xy -2.24689 4.425404) (xy -2.075917 4.334774) (xy -1.85854 4.222812) (xy -1.607442 4.096218)
+				(xy -1.559937 4.072542) (xy -0.720985 3.655135) (xy -0.353649 3.84762) (xy 0.013688 4.040105) (xy 0.365799 3.846855)
+				(xy 0.717909 3.653605)
+			)
+			(stroke
+				(width 0)
+				(type solid)
+			)
+			(fill yes)
+			(layer "F.SilkS")
+		)
+		(fp_poly
+			(pts
+				(xy -0.613824 -1.801972) (xy -0.616166 1.905) (xy -1.875771 3.033889) (xy -2.168765 3.294526) (xy -2.442611 3.534404)
+				(xy -2.688806 3.746357) (xy -2.898847 3.923218) (xy -3.06423 4.057822) (xy -3.176453 4.143001) (xy -3.225744 4.171589)
+				(xy -3.329728 4.159046) (xy -3.459808 4.116638) (xy -3.468982 4.112658) (xy -3.57083 4.050273) (xy -3.620812 3.985807)
+				(xy -3.621852 3.977484) (xy -3.627007 3.920322) (xy -3.641891 3.777558) (xy -3.665635 3.557063)
+				(xy -3.697369 3.26671) (xy -3.736225 2.914372) (xy -3.781331 2.507921) (xy -3.831818 2.05523) (xy -3.886818 1.564171)
+				(xy -3.94546 1.042617) (xy -3.97463 0.783894) (xy -4.034663 0.251248) (xy -4.091478 -0.254107) (xy -4.144206 -0.724371)
+				(xy -4.191979 -1.151748) (xy -4.233931 -1.528438) (xy -4.269193 -1.846644) (xy -4.296898 -2.098567)
+				(xy -4.316179 -2.276409) (xy -4.326168 -2.372373) (xy -4.327407 -2.387122) (xy -4.291249 -2.427564)
+				(xy -4.184215 -2.525473) (xy -4.00847 -2.679028) (xy -3.766178 -2.886407) (xy -3.459503 -3.145788)
+				(xy -3.090609 -3.455348) (xy -2.661659 -3.813266) (xy -2.174818 -4.21772) (xy -1.63225 -4.666888)
+				(xy -1.036118 -5.158947) (xy -1.000097 -5.188638) (xy -0.611482 -5.508942)
+			)
+			(stroke
+				(width 0)
+				(type solid)
+			)
+			(fill yes)
+			(layer "F.SilkS")
+		)
+		(fp_poly
+			(pts
+				(xy 0.74262 -5.401681) (xy 0.804774 -5.34994) (xy 0.931648 -5.24465) (xy 1.115484 -5.09224) (xy 1.348524 -4.899136)
+				(xy 1.623012 -4.671766) (xy 1.931188 -4.416557) (xy 2.265296 -4.139935) (xy 2.600583 -3.862395)
+				(xy 2.94701 -3.574849) (xy 3.270238 -3.304989) (xy 3.563213 -3.058816) (xy 3.818882 -2.842332) (xy 4.030188 -2.661539)
+				(xy 4.19008 -2.522437) (xy 4.291503 -2.431028) (xy 4.327403 -2.393315) (xy 4.327407 -2.393222) (xy 4.322249 -2.340835)
+				(xy 4.307354 -2.202768) (xy 4.283593 -1.986813) (xy 4.251838 -1.700764) (xy 4.212958 -1.352415)
+				(xy 4.167824 -0.949558) (xy 4.117307 -0.499988) (xy 4.062279 -0.011498) (xy 4.003608 0.50812) (xy 3.974713 0.763617)
+				(xy 3.91453 1.296672) (xy 3.857583 1.803365) (xy 3.804748 2.275767) (xy 3.756899 2.705944) (xy 3.71491 3.085966)
+				(xy 3.679657 3.407901) (xy 3.652014 3.663817) (xy 3.632856 3.845782) (xy 3.623058 3.945865) (xy 3.621935 3.962239)
+				(xy 3.581767 4.027171) (xy 3.482851 4.098076) (xy 3.357403 4.156925) (xy 3.237636 4.18569) (xy 3.221575 4.186296)
+				(xy 3.174013 4.155896) (xy 3.064932 4.069384) (xy 2.902547 3.933793) (xy 2.695073 3.756154) (xy 2.450724 3.543501)
+				(xy 2.177716 3.302865) (xy 1.889138 3.045648) (xy 0.616231 1.905) (xy 0.613856 -1.803348) (xy 0.611481 -5.511695)
+			)
+			(stroke
+				(width 0)
+				(type solid)
+			)
+			(fill yes)
+			(layer "F.SilkS")
+		)
+		(embedded_fonts no)
+	)
 	(footprint "PCM_SparkFun-LED:LED_0603_1608Metric"
 		(locked yes)
@@
 		(layer "Edge.Cuts")
 	)
+	(gr_text "BY DASHIELL RUSSELL"
+		(at 131.75 142.85 0)
+		(layer "F.Cu")
+		(effects
+			(font
+				(size 1 1)
+				(thickness 0.2)
+				(bold yes)
+			)
+		)
+	)
+	(gr_text "PULL PIN, DISTRUBUTION \nAND MONITORING BOARD"
+		(at 131.9 139.05 0)
+		(layer "F.Cu")
+		(effects
+			(font
+				(size 1.5 1.5)
+				(thickness 0.3)
+				(bold yes)
+			)
+		)
+	)
+	(gr_text "UNSW AURC BMS"
+		(at 131.85 134.7 0)
+		(layer "F.Cu" knockout)
+		(effects
+			(font
+				(size 2 2)
+				(thickness 0.3)
+				(bold yes)
+			)
+		)
+	)
+	(gr_text "BY DASHIELL RUSSELL"
+		(at 131.75 142.85 0)
+		(layer "F.Mask")
+		(effects
+			(font
+				(size 1 1)
+				(thickness 0.2)
+				(bold yes)
+			)
+		)
+	)
+	(gr_text "PULL PIN, DISTRUBUTION \nAND MONITORING BOARD"
+		(at 131.9 139.05 0)
+		(layer "F.Mask")
+		(effects
+			(font
+				(size 1.5 1.5)
+				(thickness 0.3)
+				(bold yes)
+			)
+		)
+	)
+	(gr_text "UNSW AURC BMS"
+		(at 131.85 134.7 0)
+		(layer "F.Mask" knockout)
+		(effects
+			(font
+				(size 2 2)
+				(thickness 0.3)
+				(bold yes)
+			)
+		)
+	)
 	(gr_text "ERROR"
