File: board2_monitor/board2_monitor.kicad_pcb (KiCad board)
At the start: 4 copper layers, 76 x 90 mm, 84 parts, among them J1 Conn_02x04_Odd_Even, J2 Conn_02x04_Odd_Even, J3 Conn_01x04, J4 Screw_Terminal_01x08, SW1 WAKE, U1 IS31FL3731-SA

Commit message: connector fixes to the boards - swapped headers with sockets and vice versa. had to adjust the schematics too but no big changes, everything still connected appropriately
Parts:
- J1, J2: footprint Connector_PinSocket_2.54mm:PinSocket_2x04_P2.54mm_Vertical -> Connector_PinHeader_2.54mm:PinHeader_2x04_P2.54mm_Vertical; moved to B.Cu
- J3: footprint Connector_PinSocket_2.54mm:PinSocket_1x04_P2.54mm_Vertical -> Connector_PinHeader_2.54mm:PinHeader_1x04_P2.54mm_Vertical; moved to B.Cu
- turned J1 to 90 degrees
- turned J2 to 90 degrees
- turned J3 to 90 degrees
