File: board2_monitor/board2_monitor.kicad_pcb (KiCad board)
At the start: 4 copper layers, 76 x 90 mm, 84 parts, among them J1 Conn_02x04_Odd_Even, J2 Conn_02x04_Odd_Even, J3 Conn_01x04, J4 Screw_Terminal_01x08, SW1 WAKE, U1 IS31FL3731-SA

Commit message: board2_monitor: routing updates (+25 segments)
Co-Authored-By: Claude Fable 5 <noreply@anthropic.com>
Routing:
- net /CA1: track 64.6 -> 82.6 mm
- net GND: track 7.06 -> 15.0 mm, vias 1 -> 3
- net /SCL: track 39.0 -> 40.8 mm
- net /CA2: track 81.7 -> 82.4 mm
Changed lines of the file:
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@@
 	)
 	(segment
+		(start 129.225 69)
+		(end 129.225 71.155456)
+		(width 0.3)
+		(layer "F.Cu")
+		(net "/CA1")
+	)
+	(segment
+		(start 127.990456 72.39)
+		(end 117.96 72.39)
+		(width 0.3)
+		(layer "F.Cu")
+		(net "/CA1")
+	)
+	(segment
 		(start 119.25 88.75)
 		(end 118.2975 88.75)
@@
 	)
 	(segment
+		(start 129.225 71.155456)
+		(end 127.990456 72.39)
+		(width 0.3)
+		(layer "F.Cu")
+		(net "/CA1")
+	)
+	(segment
 		(start 145.25 88.75)
 		(end 144.2975 88.75)
@@
 	)
 	(segment
+		(start 117.96 72.39)
+		(end 115.05 75.3)
+		(width 0.3)
+		(layer "F.Cu")
+		(net "/CA1")
+	)
+	(segment
 		(start 116.625 83.05)
 		(end 117.5475 83.05)
@@
 	)
 	(segment
+		(start 129.875 71.212563)
+		(end 129.875 69)
+		(width 0.3)
+		(layer "F.Cu")
+		(net "/CA2")
+	)
+	(segment
 		(start 123.7275 86.15)
 		(end 122.775 86.15)
@@
 	)
 	(segment
+		(start 119.25 74.825001)
+		(end 121.185001 72.89)
+		(width 0.3)
+		(layer "F.Cu")
+		(net "/CA2")
+	)
+	(segment
 		(start 136.5875 86.15)
 		(end 135.635 86.15)
@@
 	)
 	(segment
-		(start 119.25 75.3)
-		(end 122.175 72.375)
-		(width 0.3)
-		(layer "F.Cu")
-		(net "/CA2")
-	)
-	(segment
-		(start 129.875 70.505456)
-		(end 129.875 69)
-		(width 0.3)
-		(layer "F.Cu")
-		(net "/CA2")
-	)
-	(segment
-		(start 128.005456 72.375)
-		(end 129.875 70.505456)
-		(width 0.3)
-		(layer "F.Cu")
-		(net "/CA2")
-	)
-	(segment
 		(start 120.825 84.6)
 		(end 121.7475 84.6)
@@
 	)
 	(segment
+		(start 119.25 75.3)
+		(end 119.25 74.825001)
+		(width 0.3)
+		(layer "F.Cu")
+		(net "/CA2")
+	)
+	(segment
 		(start 120.825 88.75)
 		(end 121.7475 88.75)
@@
 	)
 	(segment
-		(start 122.175 72.375)
-		(end 128.005456 72.375)
+		(start 128.197563 72.89)
+		(end 129.875 71.212563)
 		(width 0.3)
 		(layer "F.Cu")
@@
 	)
 	(segment
+		(start 121.185001 72.89)
+		(end 128.197563 72.89)
+		(width 0.3)
+		(layer "F.Cu")
+		(net "/CA2")
+	)
+	(segment
 		(start 120.825 79.95)
 		(end 121.7475 79.95)
@@
 	)
 	(segment
-		(start 128.212562 72.875)
-		(end 130.525 70.562562)
-		(width 0.3)
-		(layer "F.Cu")
-		(net "/CA3")
-	)
-	(segment
 		(start 125.3025 76.86)
 		(end 126.215 76.86)
@@
 	)
 	(segment
-		(start 123.7275 75.3)
-		(end 126.1525 72.875)
-		(width 0.3)
-		(layer "F.Cu")
-		(net "/CA3")
-	)
-	(segment
 		(start 127.9275 84.6)
 		(end 126.975 84.6)
@@
 	)
 	(segment
+		(start 125.6375 73.39)
+		(end 128.40467 73.39)
+		(width 0.3)
+		(layer "F.Cu")
+		(net "/CA3")
+	)
+	(segment
 		(start 125.3025 84.6)
 		(end 126.225 84.6)
@@
 	)
 	(segment
+		(start 123.7275 75.3)
+		(end 125.6375 73.39)
+		(width 0.3)
+		(layer "F.Cu")
+		(net "/CA3")
+	)
+	(segment
+		(start 128.40467 73.39)
+		(end 130.525 71.26967)
+		(width 0.3)
+		(layer "F.Cu")
+		(net "/CA3")
+	)
+	(segment
 		(start 125.3025 88.75)
 		(end 126.225 88.75)
@@
 	)
 	(segment
-		(start 130.525 70.562562)
-		(end 130.525 69)
-		(width 0.3)
-		(layer "F.Cu")
-		(net "/CA3")
-	)
-	(segment
 		(start 125.3025 83.05)
 		(end 126.225 83.05)
@@
 	)
 	(segment
+		(start 130.525 71.26967)
+		(end 130.525 69)
+		(width 0.3)
+		(layer "F.Cu")
+		(net "/CA3")
+	)
+	(segment
 		(start 119.25 86.15)
 		(end 118.2975 86.15)
@@
 	)
 	(segment
-		(start 126.1525 72.875)
-		(end 128.212562 72.875)
-		(width 0.3)
-		(layer "F.Cu")
-		(net "/CA3")
-	)
-	(segment
 		(start 126.215 76.86)
 		(end 126.225 76.85)
@@
 	)
 	(segment
-		(start 127.9275 73.867169)
-		(end 131.175 70.619668)
-		(width 0.3)
-		(layer "F.Cu")
-		(net "/CA4")
-	)
-	(segment
 		(start 136.5875 83.05)
 		(end 135.635 83.05)
@@
 	)
 	(segment
-		(start 131.175 70.619668)
+		(start 129.5025 81.5)
+		(end 130.425 81.5)
+		(width 0.2)
+		(locked yes)
+		(layer "F.Cu")
+		(net "/CA4")
+	)
+	(segment
+		(start 131.175 71.326776)
 		(end 131.175 69)
 		(width 0.3)
@@
 	)
 	(segment
-		(start 129.5025 81.5)
-		(end 130.425 81.5)
-		(width 0.2)
-		(locked yes)
+		(start 127.9275 74.574276)
+		(end 131.175 71.326776)
+		(width 0.3)
 		(layer "F.Cu")
 		(net "/CA4")
@@
 	)
 	(segment
+		(start 127.9275 75.3)
+		(end 127.9275 74.574276)
+		(width 0.3)
+		(layer "F.Cu")
+		(net "/CA4")
+	)
+	(segment
 		(start 129.5025 84.6)
 		(end 130.425 84.6)
@@
 	)
 	(segment
-		(start 127.9275 75.3)
-		(end 127.9275 73.867169)
-		(width 0.3)
-		(layer "F.Cu")
-		(net "/CA4")
-	)
-	(segment
 		(start 129.5025 88.75)
 		(end 130.425 88.75)
@@
 	)
 	(segment
+		(start 131.175 62)
+		(end 131.175 63.357)
+		(width 0.5)
+		(layer "F.Cu")
+		(net "GND")
+	)
+	(segment
 		(start 130.855 56.45)
 		(end 132.055 57.65)
@@
 	)
 	(segment
+		(start 126.625 67.443)
+		(end 126.492 67.31)
+		(width 0.5)
+		(layer "F.Cu")
+		(net "GND")
+	)
+	(segment
+		(start 126.625 70.425)
+		(end 127.5 71.3)
+		(width 0.5)
+		(layer "F.Cu")
+		(net "GND")
+	)
+	(segment
 		(start 130.05 56.45)
 		(end 130.855 56.45)
@@
 	)
 	(segment
+		(start 131.175 63.357)
+		(end 131.318 63.5)
+		(width 0.5)
+		(layer "F.Cu")
+		(net "GND")
+	)
+	(segment
 		(start 129.3 56.45)
 		(end 128.05 57.7)
@@
 		(net "GND")
 	)
+	(segment
+		(start 127.275 68.093)
+		(end 126.492 67.31)
+		(width 0.5)
+		(layer "F.Cu")
+		(net "GND")
+	)
+	(segment
+		(start 126.625 69)
+		(end 126.625 70.425)
+		(width 0.5)
+		(layer "F.Cu")
+		(net "GND")
+	)
+	(segment
+		(start 126.625 69)
+		(end 126.625 67.443)
+		(width 0.5)
+		(layer "F.Cu")
+		(net "GND")
+	)
+	(segment
+		(start 127.275 69)
+		(end 127.275 68.093)
+		(width 0.5)
+		(layer "F.Cu")
+		(net "GND")
+	)
 	(via
 		(at 130.05 56.45)
@@
 		(net "GND")
 	)
+	(via
+		(at 131.318 63.5)
+		(size 0.6)
+		(drill 0.3)
+		(layers "F.Cu" "B.Cu")
+		(net "GND")
+	)
+	(via
+		(at 126.492 67.31)
+		(size 0.6)
+		(drill 0.3)
+		(layers "F.Cu" "B.Cu")
+		(net "GND")
+	)
 	(segment
 		(start 142.32254 115.15)
@@
 	)
 	(segment
-		(start 127.925 69)
-		(end 127.925 67.475)
+		(start 127.925 67.475)
+		(end 127.925 69)
 		(width 0.3)
 		(layer "F.Cu")
@@
 	)
 	(segment
-		(start 127.925 67.475)
-		(end 128.1 67.3)
+		(start 128.1 67.3)
+		(end 127.925 67.475)
 		(width 0.3)
 		(layer "F.Cu")
@@
 		(net "/SDA")
 	)
+	(segment
+		(start 129.094412 67.4)
+		(end 129.1 67.4)
+		(width 0.5)
+		(layer "F.Cu")
+		(net "/SCL")
+	)
+	(segment
+		(start 129.1 67.4)
+		(end 128.575 67.925)
+		(width 0.3)
+		(layer "F.Cu")
+		(net "/SCL")
+	)
+	(segment
+		(start 128.575 67.925)
+		(end 128.575 69)
+		(width 0.3)
+		(layer "F.Cu")
+		(net "/SCL")
+	)
 	(via
