File: board1_power/board1_power.kicad_pcb (KiCad board)
At the start: 0 parts

Commit message: board1_power: PCB footprint placement + layout updates
Co-Authored-By: Claude Opus 4.8 (1M context) <noreply@anthropic.com>
Parts:
- added C1: 10uF, Capacitor_SMD:C_0805_2012Metric, B.Cu at (262.6, 45.1)
- added C10: 10uf/25V, Capacitor_SMD:C_1206_3216Metric, B.Cu at (260.4, 61.9)
- added C11: 0.1uF, Capacitor_SMD:C_0603_1608Metric, B.Cu at (253.4, 47.0)
- added C12: 47nF, Capacitor_SMD:C_0805_2012Metric, B.Cu at (261.0, 55.7)
- added C13: 22uF, Capacitor_SMD:C_1206_3216Metric, B.Cu at (255.9, 52.3)
- added C14: 6.8uF/25V, Capacitor_SMD:C_0805_2012Metric, B.Cu at (261.0, 59.7)
- added C15: 4.7uF, Capacitor_SMD:C_0805_2012Metric, B.Cu at (261.0, 57.7)
- added C16: 0.1uF, Capacitor_SMD:C_0603_1608Metric, B.Cu at (248.1, 66.1)
- added C17: 10uf/25V, Capacitor_SMD:C_1206_3216Metric, B.Cu at (241.9, 61.9)
- added C18: 0.1uF, Capacitor_SMD:C_0603_1608Metric, B.Cu at (234.9, 47.0)
- added C19: 47nF, Capacitor_SMD:C_0805_2012Metric, B.Cu at (242.5, 55.7)
- added C20: 22uF, Capacitor_SMD:C_1206_3216Metric, B.Cu at (237.4, 52.3)
- added C21: 6.8uF/25V, Capacitor_SMD:C_0805_2012Metric, B.Cu at (242.5, 59.7)
- added C22: 4.7uF, Capacitor_SMD:C_0805_2012Metric, B.Cu at (242.5, 57.7)
- added C23: 0.1uF, Capacitor_SMD:C_0603_1608Metric, B.Cu at (229.6, 66.1)
- added C24: 10uf/25V, Capacitor_SMD:C_1206_3216Metric, B.Cu at (223.4, 61.9)
- added C25: 0.1uF, Capacitor_SMD:C_0603_1608Metric, B.Cu at (216.4, 47.0)
- added C26: 47nF, Capacitor_SMD:C_0805_2012Metric, B.Cu at (224.0, 55.7)
- added C27: 22uF, Capacitor_SMD:C_1206_3216Metric, B.Cu at (218.9, 52.3)
- added C28: 6.8uF/25V, Capacitor_SMD:C_0805_2012Metric, B.Cu at (224.0, 59.7)
- added C29: 4.7uF, Capacitor_SMD:C_0805_2012Metric, B.Cu at (224.0, 57.7)
- added C3: 1uF, Capacitor_SMD:C_0603_1608Metric, B.Cu at (188.8, 77.4)
- added C30: 0.1uF, Capacitor_SMD:C_0603_1608Metric, B.Cu at (211.1, 66.1)
- added C31: 10uf/25V, Capacitor_SMD:C_1206_3216Metric, B.Cu at (204.9, 61.9)
- added C32: 0.1uF, Capacitor_SMD:C_0603_1608Metric, B.Cu at (197.9, 47.0)
- added C33: 47nF, Capacitor_SMD:C_0805_2012Metric, B.Cu at (205.5, 55.7)
- added C34: 22uF, Capacitor_SMD:C_1206_3216Metric, B.Cu at (200.4, 52.3)
- added C35: 6.8uF/25V, Capacitor_SMD:C_0805_2012Metric, B.Cu at (205.5, 59.7)
- added C36: 4.7uF, Capacitor_SMD:C_0805_2012Metric, B.Cu at (205.5, 57.7)
- added C37: 0.1uF, Capacitor_SMD:C_0603_1608Metric, B.Cu at (192.6, 66.1)
- added C38: 1uF, Capacitor_SMD:C_0805_2012Metric, B.Cu at (211.6, 77.0)
- added C4: 10uF, Capacitor_SMD:C_0805_2012Metric, B.Cu at (186.9, 77.2)
- added C5: 100nF, Capacitor_SMD:C_0805_2012Metric, B.Cu at (184.9, 77.2)
- added C7: 1uF, Capacitor_SMD:C_0805_2012Metric, B.Cu at (211.6, 74.9)
- added C8: 47uF/ 25V, Capacitor_SMD:CP_Elec_6.3x5.4, B.Cu at (235.5, 101.0)
- added C9: 1uF/25V, Capacitor_SMD:C_0603_1608Metric, B.Cu at (224.9, 98.2)
- added D1: LED, LED_SMD:LED_0603_1608Metric, B.Cu at (187.2, 102.0)
- added D10: SK6812, LED_SMD:LED_SK6812_PLCC4_5.0x5.0mm_P3.2mm, B.Cu at (202.2, 45.8)
- added D12: MMBD4448HCQW, Package_TO_SOT_SMD:SOT-353_SC-70-5, B.Cu at (207.9, 80.1)
- added D2: PD_GOOD, PCM_SparkFun-LED:LED_0603_1608Metric_Green, B.Cu at (224.9, 102.8)
- added D3: LED, LED_SMD:LED_0603_1608Metric, B.Cu at (255.8, 62.6)
- added D4: SK6812, LED_SMD:LED_SK6812_PLCC4_5.0x5.0mm_P3.2mm, B.Cu at (257.8, 45.8)
- added D5: LED, LED_SMD:LED_0603_1608Metric, B.Cu at (237.3, 62.6)
- added D6: SK6812, LED_SMD:LED_SK6812_PLCC4_5.0x5.0mm_P3.2mm, B.Cu at (239.2, 45.8)
- added D7: LED, LED_SMD:LED_0603_1608Metric, B.Cu at (218.8, 62.6)
- added D8: SK6812, LED_SMD:LED_SK6812_PLCC4_5.0x5.0mm_P3.2mm, B.Cu at (220.8, 45.8)
- added D9: LED, LED_SMD:LED_0603_1608Metric, B.Cu at (200.3, 62.6)
- added F1: Polyfuse, Fuse:Fuse_1812_4532Metric, B.Cu at (250.0, 45.9)
- added F2: Polyfuse, Fuse:Fuse_1812_4532Metric, B.Cu at (231.5, 45.9)
- added F3: Polyfuse, Fuse:Fuse_1812_4532Metric, B.Cu at (213.0, 45.9)
- added F4: Polyfuse, Fuse:Fuse_1812_4532Metric, B.Cu at (194.5, 45.9)
- added J1: Conn_02x04_Odd_Even, Connector_PinHeader_2.54mm:PinHeader_2x04_P2.54mm_Horizontal, F.Cu at (243.7, 32.1)
- added J2: Conn_01x04, Connector_PinHeader_2.54mm:PinHeader_1x04_P2.54mm_Horizontal, F.Cu at (231.0, 29.6)
- added J3: USB_C_Receptacle_USB2.0_16P, Connector_USB:USB_C_Receptacle_GCT_USB4105-xx-A_16P_TopMnt_Horizontal, B.Cu at (226.8, 113.2)
- added J4: POWER_OFF_HEADER, Connector_PinHeader_2.54mm:PinHeader_1x02_P2.54mm_Horizontal, B.Cu at (206.9, 106.4)
- added J5: BH-18650-A1BJ024, BMS:BH-18650-A1BJ024, F.Cu at (226.8, 73.9)
- added JP1: Boot, TestPoint:TestPoint_2Pads_Pitch2.54mm_Drill0.8mm, B.Cu at (193.4, 101.3)
- added L1: SRP5030CA-2R2M, BMS:IND-SMD_L5.5-W5.3, B.Cu at (259.9, 51.7)
- added L2: SRP5030CA-2R2M, BMS:IND-SMD_L5.5-W5.3, B.Cu at (241.4, 51.7)
- added L3: SRP5030CA-2R2M, BMS:IND-SMD_L5.5-W5.3, B.Cu at (222.9, 51.7)
- added L4: SRP5030CA-2R2M, BMS:IND-SMD_L5.5-W5.3, B.Cu at (204.4, 51.7)
- added Q1: DMG2305UX, Package_TO_SOT_SMD:SOT-23, B.Cu at (247.7, 58.4)
- added Q2: SI4920DY, BMS:SOIC-8_L4.9-W3.9-P1.27-LS6.2-BL, B.Cu at (259.4, 67.5)
- added Q3: DMG2305UX, Package_TO_SOT_SMD:SOT-23, B.Cu at (229.2, 58.4)
- added Q4: SI4920DY, BMS:SOIC-8_L4.9-W3.9-P1.27-LS6.2-BL, B.Cu at (240.9, 67.5)
- added Q5: DMG2305UX, Package_TO_SOT_SMD:SOT-23, B.Cu at (210.7, 58.4)
- added Q6: SI4920DY, BMS:SOIC-8_L4.9-W3.9-P1.27-LS6.2-BL, B.Cu at (222.4, 67.5)
- added Q7: DMG2305UX, Package_TO_SOT_SMD:SOT-23, B.Cu at (192.2, 58.4)
- added Q8: SI4920DY, BMS:SOIC-8_L4.9-W3.9-P1.27-LS6.2-BL, B.Cu at (203.9, 67.5)
- added Q9: 2N7002, Package_TO_SOT_SMD:SOT-23, B.Cu at (203.5, 75.8)
- added R1: 10K, Resistor_SMD:R_0603_1608Metric, B.Cu at (211.3, 80.8)
- added R11: 24K, Resistor_SMD:R_0603_1608Metric, B.Cu at (224.9, 104.3)
- added R12: 1K, Resistor_SMD:R_0805_2012Metric, B.Cu at (226.8, 94.9)
- added R13: 10K, Resistor_SMD:R_0603_1608Metric, B.Cu at (225.7, 100.5)
- added R14: 1K, Resistor_SMD:R_0603_1608Metric, B.Cu at (224.1, 100.5)
- added R15: 30.3R, Resistor_SMD:R_0603_1608Metric, B.Cu at (251.7, 59.9)
- added R16: 1K, Resistor_SMD:R_0603_1608Metric, B.Cu at (257.3, 62.6)
- added R17: 360R, Resistor_SMD:R_0603_1608Metric, B.Cu at (251.7, 61.4)
- added R18: 5.24R, Resistor_SMD:R_0603_1608Metric, B.Cu at (251.7, 58.4)
- added R19: 100K, Resistor_SMD:R_0603_1608Metric, B.Cu at (251.7, 56.9)
- added R2: 4.7K, Resistor_SMD:R_0603_1608Metric, B.Cu at (198.7, 77.4)
- added R20: 0R, Resistor_SMD:R_2010_5025Metric, B.Cu at (251.7, 52.1)
- added R21: 100R, Resistor_SMD:R_0603_1608Metric, B.Cu at (248.1, 67.6)
- added R22: 100k, PCM_SparkFun-Resistor:R_0603_1608Metric, B.Cu at (247.3, 61.0)
- added R23: 0R, Resistor_SMD:R_2010_5025Metric, B.Cu at (248.2, 52.1)
- added R24: 2K, Resistor_SMD:R_0603_1608Metric, B.Cu at (253.8, 69.3)
- added R25: 30.3R, Resistor_SMD:R_0603_1608Metric, B.Cu at (233.2, 59.9)
- added R26: 1K, Resistor_SMD:R_0603_1608Metric, B.Cu at (238.8, 62.6)
- added R27: 360R, Resistor_SMD:R_0603_1608Metric, B.Cu at (233.2, 61.4)
- added R28: 5.24R, Resistor_SMD:R_0603_1608Metric, B.Cu at (233.2, 58.4)
- added R29: 100K, Resistor_SMD:R_0603_1608Metric, B.Cu at (233.2, 56.9)
- added R3: 4.7K, Resistor_SMD:R_0603_1608Metric, B.Cu at (205.9, 84.8)
- added R30: 0R, Resistor_SMD:R_2010_5025Metric, B.Cu at (233.2, 52.1)
- added R31: 100R, Resistor_SMD:R_0603_1608Metric, B.Cu at (229.6, 67.6)
- added R32: 100k, PCM_SparkFun-Resistor:R_0603_1608Metric, B.Cu at (228.8, 61.0)
- added R33: 0R, Resistor_SMD:R_2010_5025Metric, B.Cu at (229.7, 52.1)
- added R34: 2K, Resistor_SMD:R_0603_1608Metric, B.Cu at (235.3, 69.3)
- added R35: 30.3R, Resistor_SMD:R_0603_1608Metric, B.Cu at (214.7, 59.9)
- added R36: 1K, Resistor_SMD:R_0603_1608Metric, B.Cu at (220.3, 62.6)
- added R37: 360R, Resistor_SMD:R_0603_1608Metric, B.Cu at (214.7, 61.4)
- added R38: 5.24R, Resistor_SMD:R_0603_1608Metric, B.Cu at (214.7, 58.4)
- added R39: 100K, Resistor_SMD:R_0603_1608Metric, B.Cu at (214.7, 56.9)
- added R4: 10K, Resistor_SMD:R_0603_1608Metric, B.Cu at (190.3, 77.4)
- added R40: 0R, Resistor_SMD:R_2010_5025Metric, B.Cu at (214.7, 52.1)
- added R41: 100R, Resistor_SMD:R_0603_1608Metric, B.Cu at (211.1, 67.6)
- added R42: 100k, PCM_SparkFun-Resistor:R_0603_1608Metric, B.Cu at (210.3, 61.0)
- added R43: 0R, Resistor_SMD:R_2010_5025Metric, B.Cu at (211.2, 52.1)
- added R44: 2K, Resistor_SMD:R_0603_1608Metric, B.Cu at (216.8, 69.3)
- added R45: 30.3R, Resistor_SMD:R_0603_1608Metric, B.Cu at (196.2, 59.9)
- added R46: 1K, Resistor_SMD:R_0603_1608Metric, B.Cu at (201.8, 62.6)
- added R47: 360R, Resistor_SMD:R_0603_1608Metric, B.Cu at (196.2, 61.4)
- added R48: 5.24R, Resistor_SMD:R_0603_1608Metric, B.Cu at (196.2, 58.4)
- added R49: 100K, Resistor_SMD:R_0603_1608Metric, B.Cu at (196.2, 56.9)
- added R5: 10K, Resistor_SMD:R_0603_1608Metric, B.Cu at (201.2, 102.0)
- added R50: 0R, Resistor_SMD:R_2010_5025Metric, B.Cu at (196.2, 52.1)
- added R51: 100R, Resistor_SMD:R_0603_1608Metric, B.Cu at (192.6, 67.6)
- added R52: 100k, PCM_SparkFun-Resistor:R_0603_1608Metric, B.Cu at (191.8, 61.0)
- added R53: 0R, Resistor_SMD:R_2010_5025Metric, B.Cu at (192.7, 52.1)
- added R54: 2K, Resistor_SMD:R_0603_1608Metric, B.Cu at (198.3, 69.3)
- added R56: 10K, Resistor_SMD:R_0603_1608Metric, B.Cu at (211.3, 79.2)
- added R57: 100K, Resistor_SMD:R_0603_1608Metric, B.Cu at (211.3, 82.5)
- added R58: 33K, Resistor_SMD:R_0603_1608Metric, B.Cu at (211.3, 84.0)
- added R59: 100K, Resistor_SMD:R_0603_1608Metric, B.Cu at (205.2, 81.4)
- added R6: 10K, Resistor_SMD:R_0603_1608Metric, B.Cu at (205.9, 86.3)
- added R60: 100K, Resistor_SMD:R_0603_1608Metric, B.Cu at (205.3, 78.0)
- added R61: 100K, Resistor_SMD:R_0603_1608Metric, B.Cu at (203.1, 78.5)
- added R7: 330R, Resistor_SMD:R_0603_1608Metric, B.Cu at (205.9, 95.2)
- added TH1: NCP18XH103, Resistor_SMD:R_0603_1608Metric, B.Cu at (254.3, 76.4)
- added TH2: NCP18XH103, Resistor_SMD:R_0603_1608Metric, B.Cu at (235.8, 76.4)
- added TH3: NCP18XH103, Resistor_SMD:R_0603_1608Metric, B.Cu at (217.3, 76.4)
- added TH4: NCP18XH103, Resistor_SMD:R_0603_1608Metric, B.Cu at (197.1, 77.4)
- added U1: ESP32-S3-WROOM-1, RF_Module:ESP32-S3-WROOM-1, B.Cu at (189.9, 89.5)
- added U10: SY6970QCC, BMS:QFN-24_L4.0-W4.0-P0.50-TL-EP2.7, B.Cu at (219.3, 57.7)
- added U11: DW01A, Package_TO_SOT_SMD:SOT-23-6, B.Cu at (214.7, 66.8)
- added U12: SY6970QCC, BMS:QFN-24_L4.0-W4.0-P0.50-TL-EP2.7, B.Cu at (200.8, 57.7)
- added U13: DW01A, Package_TO_SOT_SMD:SOT-23-6, B.Cu at (196.2, 66.8)
- added U2: TCA9548APWR, Package_SO:TSSOP-24_4.4x7.8mm_P0.65mm, B.Cu at (219.7, 86.7)
- added U3: AP2112K-3.3, Package_TO_SOT_SMD:SOT-23-5, B.Cu at (208.0, 75.9)
- added U4: USBLC6-2SC6, Package_TO_SOT_SMD:SOT-23-6, B.Cu at (221.5, 100.4)
- added U5: CH224K, BMS:ESSOP-10_L4.9-W3.9-P1.0-LS6.0-TL-EP, B.Cu at (229.0, 100.5)
- added U6: SY6970QCC, BMS:QFN-24_L4.0-W4.0-P0.50-TL-EP2.7, B.Cu at (256.3, 57.7)
- added U7: DW01A, Package_TO_SOT_SMD:SOT-23-6, B.Cu at (251.7, 66.8)
- added U8: SY6970QCC, BMS:QFN-24_L4.0-W4.0-P0.50-TL-EP2.7, B.Cu at (237.8, 57.7)
- added U9: DW01A, Package_TO_SOT_SMD:SOT-23-6, B.Cu at (233.2, 66.8)
Routing:
- net GND: track 0.00 -> 254.3 mm, vias 0 -> 44
- net /CH1_V: track 0.00 -> 203.7 mm, vias 0 -> 8
- net +3V3: track 0.00 -> 194.3 mm, vias 0 -> 10
- net VBUS: track 0.00 -> 176.5 mm, vias 0 -> 13
- net SCL: track 0.00 -> 123.5 mm, vias 0 -> 2
- net SDA: track 0.00 -> 120.5 mm, vias 0 -> 2
- net /WAKE: track 0.00 -> 114.8 mm, vias 0 -> 2
- net /RGB_DATA: track 0.00 -> 106.5 mm, vias 0 -> 2
- net /CH3_CN: track 0.00 -> 84.6 mm
- net /CH2_CN: track 0.00 -> 84.2 mm
- net /CH1_CN: track 0.00 -> 76.4 mm
- net /CH4_CN: track 0.00 -> 63.1 mm, vias 0 -> 1
- net /CH4_V: track 0.00 -> 54.3 mm
- net /CH1_SDA: track 0.00 -> 49.0 mm, vias 0 -> 2
- net /CH1_SCL: track 0.00 -> 48.6 mm, vias 0 -> 2
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- added copper zone on B.Cu, net /CH4_CN
- added copper zone on B.Cu, net /Charge_Chanel1 (FC1)/CHn_V_pre
- added copper zone on B.Cu, net /Charge_Chanel2 (FC2)/CHn_V_pre
- added copper zone on B.Cu, net /Charge_Chanel3(PYRO1)/CHn_V_pre
- added copper zone on B.Cu, net /Charge_Chanel4(PYRO2)/CHn_V_pre
- added copper zone on B.Cu, net GND
- added copper zone on In1.Cu, net GND
- added copper zone on B.Cu, net VBUS
Other:
- board outline added: 100 x 100 mm
- copper layers 0 -> 4

Commit message: board1_power: place UNSW Rocketry logo (large)
Co-Authored-By: Claude Opus 4.8 (1M context) <noreply@anthropic.com>
Parts:
- added G***: LOGO, UNSW_ROCKETRY_LIBRARY:ROCKETRY_LOGO_LARGE, F.Cu at (264.9, 91.8)
Other:
- board text added: "4 INDIPENDENT CELL 18650 CELL CHARGER"
- board text added: "BY DASHIELL RUSSELL"
- board text added: "CELL 1"
- board text added: "CELL 2"
- board text added: "CELL 3"
- board text added: "CELL 4"
- board text added: "UNSW AURC ROCKETRY BMS"
Changed lines of the file:
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@@
 		)
 	)
+	(footprint "UNSW_ROCKETRY_LIBRARY:ROCKETRY_LOGO_LARGE"
+		(layer "F.Cu")
+		(at 264.9 91.8)
+		(property "Reference" "G***"
+			(at 0 0 0)
+			(layer "F.SilkS")
+			(hide yes)
+			(effects
+				(font
+					(size 1.5 1.5)
+					(thickness 0.3)
+				)
+			)
+		)
+		(property "Value" "LOGO"
+			(at 0.75 0 0)
+			(layer "F.SilkS")
+			(hide yes)
+			(effects
+				(font
+					(size 1.5 1.5)
+					(thickness 0.3)
+				)
+			)
+		)
+		(property "Datasheet" ""
+			(at 0 0 0)
+			(layer "F.Fab")
+			(hide yes)
+			(effects
+				(font
+					(size 1.27 1.27)
+				)
+			)
+		)
+		(property "Description" ""
+			(at 0 0 0)
+			(layer "F.Fab")
+			(hide yes)
+			(effects
+				(font
+					(size 1.27 1.27)
+				)
+			)
+		)
+		(attr board_only exclude_from_pos_files exclude_from_bom)
+		(duplicate_pad_numbers_are_jumpers no)
+		(fp_poly
+			(pts
+				(xy 3.550782 9.277465) (xy 4.134121 9.570367) (xy 4.645836 9.832414) (xy 5.05706 10.0484) (xy 5.338927 10.203119)
+				(xy 5.462571 10.281365) (xy 5.465797 10.286227) (xy 5.3712 10.339738) (xy 5.108049 10.459089) (xy 4.707286 10.631721)
+				(xy 4.19985 10.845074) (xy 3.616684 11.086591) (xy 2.988727 11.343711) (xy 2.34692 11.603876) (xy 1.722204 11.854527)
+				(xy 1.145519 12.083104) (xy 0.647806 12.27705) (xy 0.260007 12.423805) (xy 0.01306 12.510809) (xy -0.060494 12.529376)
+				(xy -0.182735 12.487627) (xy -0.476217 12.374968) (xy -0.913987 12.202123) (xy -1.469095 11.979818)
+				(xy -2.114589 11.718778) (xy -2.813292 11.433913) (xy -3.51596 11.144217) (xy -4.148723 10.879282)
+				(xy -4.685836 10.650217) (xy -5.101554 10.468132) (xy -5.370131 10.344137) (xy -5.465823 10.289342)
+				(xy -5.465824 10.289287) (xy -5.374425 10.225816) (xy -5.119497 10.083197) (xy -4.729938 9.8767)
+				(xy -4.234648 9.621596) (xy -3.662527 9.333155) (xy -3.554287 9.279209) (xy -1.642751 8.328156)
+				(xy -0.805782 8.766729) (xy 0.031187 9.205301) (xy 0.833464 8.764986) (xy 1.635742 8.32467)
+			)
+			(stroke
+				(width 0)
+				(type solid)
+			)
+			(fill yes)
+			(layer "B.SilkS")
+		)
+		(fp_poly
+			(pts
+				(xy -1.398586 -4.105759) (xy -1.403923 4.340505) (xy -4.273909 6.912657) (xy -4.941489 7.506514)
+				(xy -5.565443 8.053072) (xy -6.126394 8.536003) (xy -6.604969 8.938978) (xy -6.981792 9.245669)
+				(xy -7.237488 9.439748) (xy -7.349796 9.504886) (xy -7.586723 9.476306) (xy -7.883109 9.379681)
+				(xy -7.904009 9.370612) (xy -8.136068 9.228469) (xy -8.249951 9.081584) (xy -8.252322 9.062622)
+				(xy -8.264066 8.932379) (xy -8.29798 8.607093) (xy -8.35208 8.104699) (xy -8.424387 7.443136) (xy -8.512917 6.640341)
+				(xy -8.615691 5.71425) (xy -8.730726 4.682802) (xy -8.856042 3.563933) (xy -8.989655 2.375581) (xy -9.056119 1.786087)
+				(xy -9.192905 0.572462) (xy -9.322355 -0.578978) (xy -9.442495 -1.650467) (xy -9.551346 -2.624236)
+				(xy -9.646932 -3.482518) (xy -9.727276 -4.207544) (xy -9.790402 -4.781546) (xy -9.834333 -5.186756)
+				(xy -9.857092 -5.405407) (xy -9.859916 -5.439012) (xy -9.777529 -5.531158) (xy -9.533655 -5.754243)
+				(xy -9.133224 -6.104116) (xy -8.581167 -6.576625) (xy -7.882413 -7.167618) (xy -7.041895 -7.872946)
+				(xy -6.064541 -8.688455) (xy -4.955283 -9.609996) (xy -3.719051 -10.633416) (xy -2.360775 -11.754565)
+				(xy -2.278703 -11.822214) (xy -1.39325 -12.552022)
+			)
+			(stroke
+				(width 0)
+				(type solid)
+			)
+			(fill yes)
+			(layer "B.SilkS")
+		)
+		(fp_poly
+			(pts
+				(xy 1.692044 -12.307629) (xy 1.833661 -12.189736) (xy 2.122741 -11.949836) (xy 2.541608 -11.602573)
+				(xy 3.072587 -11.16259) (xy 3.698001 -10.644531) (xy 4.400175 -10.063041) (xy 5.161434 -9.432764)
+				(xy 5.925377 -8.800395) (xy 6.714706 -8.145227) (xy 7.451175 -7.530356) (xy 8.118714 -6.969456)
+				(xy 8.701248 -6.476201) (xy 9.182707 -6.064266) (xy 9.547018 -5.747325) (xy 9.778108 -5.539053)
+				(xy 9.859905 -5.453123) (xy 9.859915 -5.452912) (xy 9.848161 -5.333549) (xy 9.814223 -5.018965)
+				(xy 9.760085 -4.526916) (xy 9.687731 -3.87516) (xy 9.599143 -3.081452) (xy 9.496307 -2.163551) (xy 9.381206 -1.139214)
+				(xy 9.255824 -0.026198) (xy 9.122145 1.157741) (xy 9.056307 1.739887) (xy 8.919182 2.954441) (xy 8.78943 4.108933)
+				(xy 8.669046 5.185291) (xy 8.560022 6.165442) (xy 8.464351 7.031314) (xy 8.384027 7.764836) (xy 8.321044 8.347936)
+				(xy 8.277393 8.762541) (xy 8.255069 8.990579) (xy 8.25251 9.027886) (xy 8.160986 9.175833) (xy 7.935609 9.337388)
+				(xy 7.649778 9.471474) (xy 7.376891 9.537014) (xy 7.340296 9.538396) (xy 7.231927 9.46913) (xy 6.983388 9.272014)
+				(xy 6.613398 8.963072) (xy 6.140672 8.558326) (xy 5.583928 8.073799) (xy 4.961883 7.525514) (xy 4.304365 6.93945)
+				(xy 1.40407 4.340505) (xy 1.398659 -4.108895) (xy 1.393248 -12.558294)
+			)
+			(stroke
+				(width 0)
+				(type solid)
+			)
+			(fill yes)
+			(layer "B.SilkS")
+		)
+		(embedded_fonts no)
+	)
 	(footprint "LED_SMD:LED_0603_1608Metric"
 		(layer "B.Cu")
@@
 		(layer "Edge.Cuts")
 	)
+	(gr_text "BY DASHIELL RUSSELL"
+		(at 264.7 106.5 0)
+		(layer "B.SilkS")
+		(effects
+			(font
+				(size 1 1)
+				(thickness 0.2)
+			)
+			(justify bottom mirror)
+		)
+	)
+	(gr_text "4 INDIPENDENT \nCELL 18650 \nCELL CHARGER "
+		(at 240.85 93.95 0)
+		(layer "B.SilkS")
+		(effects
+			(font
+				(size 1.5 1.5)
+				(thickness 0.3)
+				(bold yes)
+			)
+			(justify bottom mirror)
+		)
+	)
+	(gr_text "CELL 4"
+		(at 199.65 42.7 0)
+		(layer "B.SilkS" knockout)
+		(effects
+			(font
+				(size 2 2)
+				(thickness 0.3)
+				(bold yes)
+			)
+			(justify bottom mirror)
+		)
+	)
+	(gr_text "CELL 3"
+		(at 218.15 42.7 0)
+		(layer "B.SilkS" knockout)
+		(effects
+			(font
+				(size 2 2)
+				(thickness 0.3)
+				(bold yes)
+			)
+			(justify bottom mirror)
+		)
+	)
+	(gr_text "CELL 2"
+		(at 236.65 42.7 0)
+		(layer "B.SilkS" knockout)
+		(effects
+			(font
+				(size 2 2)
+				(thickness 0.3)
+				(bold yes)
+			)
+			(justify bottom mirror)
+		)
+	)
+	(gr_text "UNSW AURC\nROCKETRY BMS"
+		(at 240.7 85.7 0)
+		(layer "B.SilkS" knockout)
+		(effects
+			(font
+				(size 2 2)
+				(thickness 0.3)
+				(bold yes)
+			)
+			(justify bottom mirror)
+		)
+	)
+	(gr_text "CELL 1"
+		(at 255.15 42.65 0)
+		(layer "B.SilkS" knockout)
+		(effects
+			(font
+				(size 2 2)
+				(thickness 0.3)
+				(bold yes)
+			)
+			(justify bottom mirror)
+		)
+	)
 	(segment
