File: board1_power/USB_IN.kicad_sch (KiCad schematic)
At the start: 10 parts, among them J3 USB_C_Receptacle_USB2.0_16P, U4 USBLC6-2SC6, U5 CH224K

Commit message: board1_power: fix PD straps + heartbeat LED resistor
- CH224K now deterministically 12V: CFG1->GND (0R), CFG2->GND (0R),
  CFG3->VDD_PD (10k pull-up = logic 1). Previously CFG2/CFG3 floated.
- Heartbeat LED D1 now has 330R series resistor to IO2 (was direct
  GPIO->LED->GND).

Closes the two items in docs/board1_fixes_todo.md.
Parts:
- added R55: 0R, Resistor_SMD:R_0805_2012Metric, symbol Device:R
- added R62: 10k, Resistor_SMD:R_0805_2012Metric, symbol Device:R
- R11: value 24K -> 0R; footprint Resistor_SMD:R_0603_1608Metric -> Resistor_SMD:R_0805_2012Metric
Connections:
- net GND: now also R55.1
- net VDD_PD: now also R62.2
- net at U5.2 (CFG2): now also R55.2
- net at U5.3 (CFG3): now also R62.1
- no-connect marks 6 -> 4
