File: board1_power/board1_power.kicad_sch (KiCad schematic)
At the start: 30 parts, among them J1 Conn_02x04_Odd_Even, J2 Conn_01x04, J4 POWER_OFF_HEADER, J5 BH-18650-A1BJ024, Q9 2N7002, U1 ESP32-S3-WROOM-1, U2 TCA9548APWR, U3 AP2112K-3.3

Commit message: connector fixes to the boards - swapped headers with sockets and vice versa. had to adjust the schematics too but no big changes, everything still connected appropriately
Parts:
- J1: footprint Connector_PinHeader_2.54mm:PinHeader_2x04_P2.54mm_Horizontal -> Connector_PinSocket_2.54mm:PinSocket_2x04_P2.54mm_Horizontal
- J2: footprint Connector_PinHeader_2.54mm:PinHeader_1x04_P2.54mm_Horizontal -> Connector_PinSocket_2.54mm:PinSocket_1x04_P2.54mm_Horizontal
Connections:
- net CH1_V: now also J1.1 (Pin_1); no longer J1.7 (Pin_7)
- net CH2_V: now also J1.3 (Pin_3); no longer J1.5 (Pin_5)
- net CH3_V: now also J1.5 (Pin_5); no longer J1.3 (Pin_3)
- net CH4_V: now also J1.7 (Pin_7); no longer J1.1 (Pin_1)
- net GND: now also J2.1 (Pin_1); no longer J2.4 (Pin_4)
- net SCL: now also J2.3 (Pin_3); no longer J2.2 (Pin_2)
- net SDA: now also J2.4 (Pin_4); no longer J2.1 (Pin_1)
- net WAKE: now also J2.2 (Pin_2); no longer J2.3 (Pin_3)
Other:
- moved on the sheet: J2
Changed lines of the file:
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@@
 	(wire
 		(pts
-			(xy 73.66 181.61) (xy 81.915 181.61)
-		)
-		(stroke
-			(width 0)
-			(type default)
-		)
-	)
-	(wire
-		(pts
 			(xy 26.035 146.685) (xy 37.465 146.685)
 		)
@@
 	(wire
 		(pts
-			(xy 73.66 179.07) (xy 81.915 179.07)
+			(xy 73.66 179.07) (xy 82.55 179.07)
 		)
 		(stroke
@@
 	(wire
 		(pts
-			(xy 74.295 186.69) (xy 81.915 186.69)
+			(xy 74.295 186.69) (xy 82.55 186.69)
 		)
 		(stroke
@@
 	(wire
 		(pts
-			(xy 49.53 184.15) (xy 55.245 184.15)
-		)
-		(stroke
-			(width 0)
-			(type default)
-		)
-	)
-	(wire
-		(pts
 			(xy 132.08 188.595) (xy 132.08 190.5)
 		)
@@
 	(wire
 		(pts
-			(xy 81.915 184.15) (xy 74.295 184.15)
+			(xy 49.53 184.15) (xy 55.245 184.15)
+		)
+		(stroke
+			(width 0)
+			(type default)
+		)
+	)
+	(wire
+		(pts
+			(xy 74.295 184.15) (xy 82.55 184.15)
 		)
 		(stroke
@@
 	(wire
 		(pts
+			(xy 49.53 179.07) (xy 55.245 179.07)
+		)
+		(stroke
+			(width 0)
+			(type default)
+		)
+	)
+	(wire
+		(pts
 			(xy 24.13 120.65) (xy 34.29 120.65)
 		)
@@
 	(wire
 		(pts
-			(xy 145.415 60.325) (xy 145.415 55.245)
+			(xy 73.66 181.61) (xy 82.55 181.61)
 		)
 		(stroke
@@
 	(wire
 		(pts
-			(xy 132.08 169.545) (xy 132.08 178.435)
+			(xy 145.415 60.325) (xy 145.415 55.245)
 		)
 		(stroke
@@
 	(wire
 		(pts
-			(xy 95.885 99.06) (xy 101.6 99.06)
+			(xy 132.08 169.545) (xy 132.08 178.435)
 		)
 		(stroke
@@
 	(wire
 		(pts
-			(xy 241.935 65.405) (xy 249.555 65.405)
+			(xy 95.885 99.06) (xy 101.6 99.06)
 		)
 		(stroke
@@
 	(wire
 		(pts
-			(xy 97.79 76.2) (xy 101.6 76.2)
+			(xy 241.935 65.405) (xy 249.555 65.405)
 		)
 		(stroke
@@
 	(wire
 		(pts
-			(xy 127 60.325) (xy 133.35 60.325)
+			(xy 97.79 76.2) (xy 101.6 76.2)
 		)
 		(stroke
@@
 	(wire
 		(pts
-			(xy 241.935 57.785) (xy 249.555 57.785)
+			(xy 127 60.325) (xy 133.35 60.325)
 		)
 		(stroke
@@
 	(wire
 		(pts
-			(xy 248.92 111.76) (xy 260.35 111.76)
+			(xy 241.935 57.785) (xy 249.555 57.785)
 		)
 		(stroke
@@
 	(wire
 		(pts
-			(xy 49.53 181.61) (xy 55.245 181.61)
+			(xy 248.92 111.76) (xy 260.35 111.76)
 		)
 		(stroke
@@
 	(wire
 		(pts
-			(xy 248.92 127) (xy 260.35 127)
+			(xy 49.53 186.69) (xy 55.245 186.69)
 		)
 		(stroke
@@
 	(wire
 		(pts
-			(xy 24.765 179.07) (xy 36.83 179.07)
+			(xy 248.92 127) (xy 260.35 127)
 		)
 		(stroke
@@
 	(wire
 		(pts
-			(xy 34.29 73.025) (xy 24.13 73.025)
+			(xy 24.765 179.07) (xy 36.83 179.07)
 		)
 		(stroke
@@
 	(wire
 		(pts
-			(xy 111.76 86.995) (xy 111.76 88.9)
+			(xy 34.29 73.025) (xy 24.13 73.025)
 		)
 		(stroke
@@
 	(wire
 		(pts
-			(xy 114.3 71.12) (xy 130.175 71.12)
+			(xy 111.76 86.995) (xy 111.76 88.9)
 		)
 		(stroke
@@
 	(wire
 		(pts
-			(xy 113.665 167.005) (xy 120.015 167.005)
+			(xy 114.3 71.12) (xy 130.175 71.12)
 		)
 		(stroke
@@
 	(wire
 		(pts
-			(xy 118.11 133.35) (xy 121.92 133.35)
+			(xy 49.53 181.61) (xy 55.245 181.61)
 		)
 		(stroke
@@
 	(wire
 		(pts
-			(xy 217.17 121.92) (xy 228.6 121.92)
+			(xy 113.665 167.005) (xy 120.015 167.005)
 		)
 		(stroke
@@
 	(wire
 		(pts
-			(xy 49.53 179.07) (xy 55.245 179.07)
+			(xy 118.11 133.35) (xy 121.92 133.35)
 		)
 		(stroke
@@
 	(wire
 		(pts
-			(xy 49.53 186.69) (xy 55.245 186.69)
+			(xy 217.17 121.92) (xy 228.6 121.92)
 		)
 		(stroke
@@
 	(symbol
 		(lib_id "Connector_Generic:Conn_01x04")
-		(at 86.995 181.61 0)
+		(at 87.63 184.15 0)
+		(mirror x)
 		(unit 1)
 		(body_style 1)
@@
 		(in_pos_files yes)
 		(dnp no)
-		(fields_autoplaced yes)
 		(property "Reference" "J2"
-			(at 89.535 181.6099 0)
+			(at 90.17 184.1501 0)
 			(show_name no)
 			(do_not_autoplace no)
@@
 		)
 		(property "Value" "Conn_01x04"
-			(at 89.535 184.1499 0)
+			(at 90.17 181.6101 0)
 			(show_name no)
 			(do_not_autoplace no)
@@
 			)
 		)
-		(property "Footprint" "Connector_PinHeader_2.54mm:PinHeader_1x04_P2.54mm_Horizontal"
-			(at 86.995 181.61 0)
+		(property "Footprint" "Connector_PinSocket_2.54mm:PinSocket_1x04_P2.54mm_Horizontal"
+			(at 87.63 184.15 0)
 			(hide yes)
 			(show_name no)
@@
 		)
 		(property "Datasheet" ""
-			(at 86.995 181.61 0)
+			(at 87.63 184.15 0)
 			(hide yes)
 			(show_name no)
@@
 		)
 		(property "Description" "Generic connector, single row, 01x04, script generated (kicad-library-utils/schlib/autogen/connector/)"
-			(at 86.995 181.61 0)
+			(at 87.63 184.15 0)
 			(hide yes)
 			(show_name no)
@@
 	(symbol
 		(lib_id "Connector_Generic:Conn_02x04_Odd_Even")
-		(at 41.91 181.61 0)
+		(at 41.91 184.15 0)
+		(mirror x)
 		(unit 1)
 		(body_style 1)
@@
 		(dnp no)
 		(property "Reference" "J1"
-			(at 43.18 173.355 0)
+			(at 43.18 192.405 0)
 			(show_name no)
 			(do_not_autoplace no)
@@
 		)
 		(property "Value" "Conn_02x04_Odd_Even"
-			(at 43.18 175.895 0)
+			(at 43.18 189.865 0)
 			(show_name no)
 			(do_not_autoplace no)
@@
 			)
 		)
-		(property "Footprint" "Connector_PinHeader_2.54mm:PinHeader_2x04_P2.54mm_Horizontal"
-			(at 41.91 181.61 0)
+		(property "Footprint" "Connector_PinSocket_2.54mm:PinSocket_2x04_P2.54mm_Horizontal"
+			(at 41.91 184.15 0)
 			(hide yes)
 			(show_name no)
@@
 		)
 		(property "Datasheet" ""
-			(at 41.91 181.61 0)
+			(at 41.91 184.15 0)
 			(hide yes)
 			(show_name no)
@@
 		)
 		(property "Description" "Generic connector, double row, 02x04, odd/even pin numbering scheme (row 1 odd numbers, row 2 even numbers), script generated (kicad-library-utils/schlib/autogen/connector/)"
-			(at 41.91 181.61 0)
+			(at 41.91 184.15 0)
 			(hide yes)
 			(show_name no)

Commit message: board1_power: fix PD straps + heartbeat LED resistor
- CH224K now deterministically 12V: CFG1->GND (0R), CFG2->GND (0R),
  CFG3->VDD_PD (10k pull-up = logic 1). Previously CFG2/CFG3 floated.
- Heartbeat LED D1 now has 330R series resistor to IO2 (was direct
  GPIO->LED->GND).

Closes the two items in docs/board1_fixes_todo.md.
Parts:
- added R8: 330R, Resistor_SMD:R_0603_1608Metric, symbol Device:R
Connections:
- net Heartbeat LED: now also R8.2; no longer D1.2 (A)
- new net: D1.2 (A), R8.1
Changed lines of the file:
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@@
 	(wire
 		(pts
-			(xy 25.4 91.44) (xy 34.29 91.44)
+			(xy 83.82 133.35) (xy 100.33 133.35)
 		)
 		(stroke
@@
 	(wire
 		(pts
-			(xy 34.29 48.895) (xy 24.13 48.895)
+			(xy 25.4 91.44) (xy 34.29 91.44)
 		)
 		(stroke
@@
 	(wire
 		(pts
-			(xy 123.19 174.625) (xy 123.19 176.53)
+			(xy 34.29 48.895) (xy 24.13 48.895)
 		)
 		(stroke
@@
 	(wire
 		(pts
-			(xy 24.13 96.52) (xy 24.13 118.11)
+			(xy 123.19 174.625) (xy 123.19 176.53)
 		)
 		(stroke
@@
 	(wire
 		(pts
-			(xy 95.25 133.35) (xy 110.49 133.35)
+			(xy 24.13 96.52) (xy 24.13 118.11)
 		)
 		(stroke
@@
 	(wire
 		(pts
+			(xy 107.95 133.35) (xy 110.49 133.35)
+		)
+		(stroke
+			(width 0)
+			(type default)
+		)
+	)
+	(wire
+		(pts
 			(xy 30.48 123.19) (xy 34.29 123.19)
 		)
@@
 	)
 	(label "Heartbeat LED"
-		(at 95.25 133.35 0)
+		(at 83.82 133.35 0)
 		(effects
 			(font
@@
 					(unit 1)
 				)
+			)
+		)
+	)
+	(symbol
+		(lib_id "Device:R")
+		(at 104.14 133.35 270)
+		(unit 1)
+		(body_style 1)
+		(exclude_from_sim no)
+		(in_bom yes)
+		(on_board yes)
+		(in_pos_files yes)
+		(dnp no)
+		(property "Reference" "R8"
+			(at 101.6 128.905 90)
+			(show_name no)
+			(do_not_autoplace no)
+			(effects
+				(font
+					(size 1.27 1.27)
+				)
+				(justify left)
+			)
+		)
+		(property "Value" "330R"
+			(at 101.6 130.81 90)
+			(show_name no)
+			(do_not_autoplace no)
+			(effects
+				(font
+					(size 1.27 1.27)
+				)
+				(justify left)
+			)
+		)
+		(property "Footprint" "Resistor_SMD:R_0603_1608Metric"
+			(at 104.14 131.572 90)
+			(hide yes)
+			(show_name no)
+			(do_not_autoplace no)
+			(effects
+				(font
+					(size 1.27 1.27)
+				)
+			)
+		)
+		(property "Datasheet" ""
+			(at 104.14 133.35 0)
+			(hide yes)
+			(show_name no)
+			(do_not_autoplace no)
+			(effects
+				(font
+					(size 1.27 1.27)
+				)
+			)
+		)
+		(property "Description" "Resistor"
+			(at 104.14 133.35 0)
+			(hide yes)
+			(show_name no)
+			(do_not_autoplace no)
+			(effects
+				(font
+					(size 1.27 1.27)
+				)
+			)
+		)
+		(pin "2"
+		)
+		(pin "1"
+		)
+		(instances
+			(project "board1_power"
+				(path "/0d1390b9-e848-4ad4-8bef-84851d0f73a3"
+					(reference "R8")
+					(unit 1)
+				)
