File: board3_dist/board3_dist.kicad_pcb (KiCad board)
At the start: 0 parts

Commit message: board3_dist: connector schematic capture (J1-J9) + initial footprint placement
Co-Authored-By: Claude Opus 4.8 (1M context) <noreply@anthropic.com>
Parts:
- added G***: ImageLogo, UNSW_ROCKETRY_LIBRARY:JUNO, F.Cu at (150.0, 126.7)
- added G***: LOGO, UNSW_ROCKETRY_LIBRARY:ROCKETRY_LOGO_SMALL, F.Cu at (123.0, 50.0)
- added J1: Conn_02x04_Odd_Even, Connector_PinHeader_2.54mm:PinHeader_2x04_P2.54mm_Horizontal, F.Cu at (166.9, 55.2)
- added J2: Screw_Terminal_01x02, TerminalBlock_Phoenix:TerminalBlock_Phoenix_PT-1,5-2-3.5-H_1x02_P3.50mm_Horizontal, F.Cu at (134.7, 77.6)
- added J3: Screw_Terminal_01x02, TerminalBlock_Phoenix:TerminalBlock_Phoenix_PT-1,5-2-3.5-H_1x02_P3.50mm_Horizontal, F.Cu at (143.7, 77.6)
- added J4: Screw_Terminal_01x02, TerminalBlock_Phoenix:TerminalBlock_Phoenix_PT-1,5-2-3.5-H_1x02_P3.50mm_Horizontal, F.Cu at (152.8, 77.6)
- added J5: Screw_Terminal_01x02, TerminalBlock_Phoenix:TerminalBlock_Phoenix_PT-1,5-2-3.5-H_1x02_P3.50mm_Horizontal, F.Cu at (161.8, 77.6)
- added J6: Conn_01x02, Connector_PinHeader_2.54mm:PinHeader_1x02_P2.54mm_Horizontal, F.Cu at (187.3, 63.7)
- added J7: Conn_01x02, Connector_PinHeader_2.54mm:PinHeader_1x02_P2.54mm_Horizontal, F.Cu at (187.3, 71.7)
- added J8: Conn_01x02, Connector_PinHeader_2.54mm:PinHeader_1x02_P2.54mm_Horizontal, F.Cu at (112.7, 74.3)
- added J9: Conn_01x02, Connector_PinHeader_2.54mm:PinHeader_1x02_P2.54mm_Horizontal, F.Cu at (112.7, 66.3)
Routing:
- net /CH2_V: track 0.00 -> 52.8 mm
- net /CH3_V: track 0.00 -> 51.6 mm
- net /FC2_FCMP: track 0.00 -> 43.8 mm
- net /CH1_V: track 0.00 -> 42.7 mm
- net /FC1_FCMP: track 0.00 -> 41.2 mm
- net /FC2_PYRO: track 0.00 -> 36.3 mm
- net /CH4_V: track 0.00 -> 35.5 mm
- net /FC1_PYRO: track 0.00 -> 27.7 mm
- added copper zone on B.Cu, net GND
Other:
- board outline added: 100 x 100 mm
- copper layers 0 -> 2
- board text added: "BATT 1"
- board text added: "BATT 2"
- board text added: "BATT 3"
- board text added: "BATT 4"
- board text added: "BY DASHIELL RUSSELL"
- board text added: "FC1"
- board text added: "FC2"
- board text added: "FCMP"
- board text added: "PULL PINS"
- board text added: "PYRO"
- board text added: "THERE WAS NEVER JUNO... ONLY EVER ME"
- board text added: "UNSW AURC 2026 POWER DISTRIBUTION BOARD"
