File: board3_dist/board3_dist.kicad_pcb (KiCad board)
At the start: 2 copper layers, 100 x 100 mm, 11 parts, among them J1 Conn_02x04_Odd_Even, J2 Screw_Terminal_01x02, J3 Screw_Terminal_01x02, J4 Screw_Terminal_01x02, J5 Screw_Terminal_01x02, J6 Conn_01x02, J7 Conn_01x02, J8 Conn_01x02, J9 Conn_01x02

Commit message: connector fixes to the boards - swapped headers with sockets and vice versa. had to adjust the schematics too but no big changes, everything still connected appropriately
Parts:
- J1: footprint Connector_PinHeader_2.54mm:PinHeader_2x04_P2.54mm_Horizontal -> Connector_PinSocket_2.54mm:PinSocket_2x04_P2.54mm_Horizontal
- J6, J7, J8, J9: footprint Connector_PinHeader_2.54mm:PinHeader_1x02_P2.54mm_Horizontal -> Connector_PinSocket_2.54mm:PinSocket_1x02_P2.54mm_Horizontal
- moved J1 7.62 mm to (174.5, 55.2), turned to -90 degrees
- moved J7 2.54 mm to (187.3, 74.3), turned to 180 degrees
- moved J8 2.54 mm to (112.7, 71.7), turned to 0 degrees
- moved J6 2.54 mm to (187.3, 66.3), turned to 180 degrees
- moved J9 2.54 mm to (112.7, 63.7), turned to 0 degrees
Connections:
- J1 pad 2: /CH4_V -> /CH1_V
- J1 pad 4: /CH3_V -> /CH2_V
- J1 pad 6: /CH2_V -> /CH3_V
- J1 pad 8: /CH1_V -> /CH4_V
- J6 pad 1: /FC1_PYRO -> GND
- J6 pad 2: GND -> /FC1_PYRO
- J7 pad 1: /FC1_FCMP -> GND
- J7 pad 2: GND -> /FC1_FCMP
- J8 pad 1: /FC2_FCMP -> GND
- J8 pad 2: GND -> /FC2_FCMP
- J9 pad 1: /FC2_PYRO -> GND
- J9 pad 2: GND -> /FC2_PYRO
