File: board3_dist/board3_dist.kicad_sch (KiCad schematic)
At the start: 0 parts

Commit message: board3_dist: connector schematic capture (J1-J9) + initial footprint placement
Co-Authored-By: Claude Opus 4.8 (1M context) <noreply@anthropic.com>
Parts:
- added J1: Conn_02x04_Odd_Even, Connector_PinHeader_2.54mm:PinHeader_2x04_P2.54mm_Horizontal, symbol Connector_Generic:Conn_02x04_Odd_Even
- added J2, J3, J4, J5: Screw_Terminal_01x02, TerminalBlock_Phoenix:TerminalBlock_Phoenix_PT-1,5-2-3.5-H_1x02_P3.50mm_Horizontal, symbol Connector:Screw_Terminal_01x02
- added J6, J7, J8, J9: Conn_01x02, Connector_PinHeader_2.54mm:PinHeader_1x02_P2.54mm_Horizontal, symbol Connector_Generic:Conn_01x02
Connections:
- new net CH1_V: J1.8 (Pin_8), J4.1 (Pin_1)
- new net CH2_V: J1.6 (Pin_6), J5.1 (Pin_1)
- new net CH3_V: J1.4 (Pin_4), J2.1 (Pin_1)
- new net CH4_V: J1.2 (Pin_2), J3.1 (Pin_1)
- new net FC1_FCMP: J4.2 (Pin_2), J7.1 (Pin_1)
- new net FC1_PYRO: J5.2 (Pin_2), J6.1 (Pin_1)
- new net FC2_FCMP: J3.2 (Pin_2), J8.1 (Pin_1)
- new net FC2_PRYO: J2.2 (Pin_2)
- new net FC2_PYRO: J9.1 (Pin_1)
- new net GND: J1.1 (Pin_1), J1.3 (Pin_3), J1.5 (Pin_5), J1.7 (Pin_7), J6.2 (Pin_2), J7.2 (Pin_2), J8.2 (Pin_2), J9.2 (Pin_2)
Other:
- note added: "BATTERIES"
- note added: "FC POWER CONECTORS"
- note added: "PULL PIN SCREW TERMINALS"
