File: board4_nosecone/USB_IN.kicad_sch (KiCad schematic)
At the start: 10 parts, among them J3 USB_C_Receptacle_USB2.0_16P, U4 USBLC6-2SC6, U5 CH224K

Commit message: board4_nosecone: complete schematic (ESP, cells, CFG 9V, dual holder)
- ESP32-S3 block wired: dual I2C buses (no mux), diode-OR gate, USB
  programming, RGB chain, WAKE/BOOT/RESET buttons
- CH224K strapped to 9V (CFG1/2/3 all to GND)
- BH-18650-B6AA007 dual 18650 holder: symbol added to BMS lib (5-pin,
  C1+/C1-/C2+/C2-/hidden mechanical), footprint relocated to BMS.pretty
  and renamed from misfiled UNSW_ROCKETRY_LIBRARY:BMSBH-18650-B6AA007
- BT1 placed, wired to CELL1/CELL2 nets

docs/board1_fixes_todo.md: main-board bugs found during the copy -
CFG2/CFG3 floating (PD not deterministically 12V), heartbeat LED
missing series resistor.

Known WIP: heartbeat LED (D1) on board4 still needs series resistor;
dangling wire stubs to clean; PD_GOOD LED (PG) unconnected; pull-pin
isolation break TBD. Verify in GUI ERC before layout.
Parts:
- removed R11: 24K, Resistor_SMD:R_0603_1608Metric, symbol Device:R
- added R28, R30, R32: 1K, Resistor_SMD:R_0805_2012Metric, symbol Device:R
- added R29, R31, R33: 0R, Resistor_SMD:R_0805_2012Metric, symbol Device:R
- renumbered C8 to C13, C9 to C14, D2 to D5, J3 to J5, R12 to R25, R13 to R26, R14 to R27, U4 to U5, U5 to U6
Connections:
- net GND: now also R29.2, R31.2, R33.2
- net VDD_PD: now also R28.1, R30.1, R32.1
- net CFG2: now reaches U6.2 (CFG2)
- net CFG2: now also R30.2, R31.1
- net CFG3: now reaches U6.3 (CFG3)
- net CFG3: now also R32.2, R33.1
- net CFG1: now reaches U6.9 (CFG1)
- net CFG1: now also R28.2, R29.1
- no-connect marks 6 -> 4
Other:
- note added: "9V"
- note added: "PD chip will negotiate for this voltage If it cant do this it will defualt to 5 So 12v or 5v doesent try 9"
- note added: "POWER DELIVERY TABLE"
