File: board4_nosecone/board4_nosecone.kicad_pcb (KiCad board)
At the start: 2 copper layers, 0 parts

Commit message: board4_nosecone: complete schematic (ESP, cells, CFG 9V, dual holder)
- ESP32-S3 block wired: dual I2C buses (no mux), diode-OR gate, USB
  programming, RGB chain, WAKE/BOOT/RESET buttons
- CH224K strapped to 9V (CFG1/2/3 all to GND)
- BH-18650-B6AA007 dual 18650 holder: symbol added to BMS lib (5-pin,
  C1+/C1-/C2+/C2-/hidden mechanical), footprint relocated to BMS.pretty
  and renamed from misfiled UNSW_ROCKETRY_LIBRARY:BMSBH-18650-B6AA007
- BT1 placed, wired to CELL1/CELL2 nets

docs/board1_fixes_todo.md: main-board bugs found during the copy -
CFG2/CFG3 floating (PD not deterministically 12V), heartbeat LED
missing series resistor.

Known WIP: heartbeat LED (D1) on board4 still needs series resistor;
dangling wire stubs to clean; PD_GOOD LED (PG) unconnected; pull-pin
isolation break TBD. Verify in GUI ERC before layout.
Parts:
- added BT1: BH-18650-B6AA007, BMS:BH-18650-B6AA007, F.Cu at (113.3, 60.2)
- added C1: 1uF, Capacitor_SMD:C_0603_1608Metric, F.Cu at (202.9, 28.6)
- added C10: 4.7uF, Capacitor_SMD:C_0805_2012Metric, F.Cu at (195.7, 57.0)
- added C11: 0.1uF, Capacitor_SMD:C_0603_1608Metric, F.Cu at (183.4, 52.3)
- added C12: 0.1uF, Capacitor_SMD:C_0603_1608Metric, F.Cu at (213.6, 49.1)
- added C13: 47uF/ 25V, Capacitor_SMD:CP_Elec_6.3x5.4, F.Cu at (191.0, 29.7)
- added C14: 1uF/25V, Capacitor_SMD:C_0603_1608Metric, F.Cu at (175.4, 33.0)
- added C15: 10uf/25V, Capacitor_SMD:C_1206_3216Metric, F.Cu at (199.8, 75.0)
- added C16: 47nF, Capacitor_SMD:C_0805_2012Metric, F.Cu at (193.6, 75.7)
- added C17: 22uF, Capacitor_SMD:C_1206_3216Metric, F.Cu at (185.8, 76.2)
- added C18: 6.8uF/25V, Capacitor_SMD:C_0805_2012Metric, F.Cu at (197.6, 75.7)
- added C19: 4.7uF, Capacitor_SMD:C_0805_2012Metric, F.Cu at (195.6, 75.7)
- added C2: 10uF, Capacitor_SMD:C_0805_2012Metric, F.Cu at (202.8, 25.2)
- added C20: 0.1uF, Capacitor_SMD:C_0603_1608Metric, F.Cu at (183.3, 71.0)
- added C21: 0.1uF, Capacitor_SMD:C_0603_1608Metric, F.Cu at (213.8, 66.6)
- added C3: 100nF, Capacitor_SMD:C_0805_2012Metric, F.Cu at (202.8, 23.1)
- added C4: 1uF, Capacitor_SMD:C_0805_2012Metric, F.Cu at (242.0, 39.8)
- added C5: 1uF, Capacitor_SMD:C_0805_2012Metric, F.Cu at (242.0, 37.8)
- added C6: 10uf/25V, Capacitor_SMD:C_1206_3216Metric, F.Cu at (199.9, 56.3)
- added C7: 47nF, Capacitor_SMD:C_0805_2012Metric, F.Cu at (193.7, 57.0)
- added C8: 22uF, Capacitor_SMD:C_1206_3216Metric, F.Cu at (185.9, 57.5)
- added C9: 6.8uF/25V, Capacitor_SMD:C_0805_2012Metric, F.Cu at (197.7, 57.0)
- added D1: LED, LED_SMD:LED_0603_1608Metric, F.Cu at (227.3, 27.1)
- added D2: MMBD4448HCQW, Package_TO_SOT_SMD:SOT-353_SC-70-5, F.Cu at (254.6, 41.1)
- added D3: LED, LED_SMD:LED_0603_1608Metric, F.Cu at (199.7, 52.4)
- added D4: SK6812, LED_SMD:LED_SK6812_PLCC4_5.0x5.0mm_P3.2mm, F.Cu at (212.3, 53.5)
- added D5: PD_GOOD, PCM_SparkFun-LED:LED_0603_1608Metric_Green, F.Cu at (175.4, 29.9)
- added D6: LED, LED_SMD:LED_0603_1608Metric, F.Cu at (199.6, 71.1)
- added D7: SK6812, LED_SMD:LED_SK6812_PLCC4_5.0x5.0mm_P3.2mm, F.Cu at (212.6, 71.0)
- added F1: Polyfuse, Fuse:Fuse_1812_4532Metric, F.Cu at (203.2, 48.1)
- added F2: Polyfuse, Fuse:Fuse_1812_4532Metric, F.Cu at (203.1, 66.8)
- added G***: LOGO, UNSW_ROCKETRY_LIBRARY:ROCKETRY_LOGO_SMALL, F.Cu at (246.8, 84.4)
- added J1: Screw_Terminal_01x04, TerminalBlock_Phoenix:TerminalBlock_Phoenix_PT-1,5-4-3.5-H_1x04_P3.50mm_Horizontal, F.Cu at (179.9, 81.7)
- added J2: Screw_Terminal_01x02, TerminalBlock_Phoenix:TerminalBlock_Phoenix_PT-1,5-2-3.5-H_1x02_P3.50mm_Horizontal, F.Cu at (228.4, 87.5)
- added J3: Screw_Terminal_01x04, TerminalBlock_Phoenix:TerminalBlock_Phoenix_PT-1,5-4-3.5-H_1x04_P3.50mm_Horizontal, F.Cu at (177.2, 98.4)
- added J4: POWER_OFF_HEADER, Connector_PinHeader_2.54mm:PinHeader_1x02_P2.54mm_Horizontal, F.Cu at (242.6, 22.6)
- added J5: USB_C_Receptacle_USB2.0_16P, Connector_USB:USB_C_Receptacle_GCT_USB4105-xx-A_16P_TopMnt_Horizontal, F.Cu at (182.4, 19.1)
- added L1: SRP5030CA-2R2M, BMS:IND-SMD_L5.5-W5.3, F.Cu at (189.9, 57.0)
- added L2: SRP5030CA-2R2M, BMS:IND-SMD_L5.5-W5.3, F.Cu at (189.8, 75.7)
- added Q1: 2N7002, Package_TO_SOT_SMD:SOT-23, F.Cu at (247.7, 41.9)
- added Q2: DMG2305UX, Package_TO_SOT_SMD:SOT-23, F.Cu at (186.4, 46.7)
- added Q3: SI4920DY, BMS:SOIC-8_L4.9-W3.9-P1.27-LS6.2-BL, F.Cu at (179.2, 56.0)
- added Q4: DMG2305UX, Package_TO_SOT_SMD:SOT-23, F.Cu at (186.3, 65.4)
- added Q5: SI4920DY, BMS:SOIC-8_L4.9-W3.9-P1.27-LS6.2-BL, F.Cu at (179.1, 74.7)
- added R1: 4.7K, Resistor_SMD:R_0603_1608Metric, F.Cu at (209.6, 44.3)
- added R10: 10K, Resistor_SMD:R_0603_1608Metric, F.Cu at (251.2, 43.0)
- added R11: 10K, Resistor_SMD:R_0603_1608Metric, F.Cu at (254.6, 43.0)
- added R12: 100K, Resistor_SMD:R_0603_1608Metric, F.Cu at (254.6, 39.2)
- added R13: 33K, Resistor_SMD:R_0603_1608Metric, F.Cu at (256.9, 39.9)
- added R14: 100K, Resistor_SMD:R_0603_1608Metric, F.Cu at (251.2, 41.1)
- added R15: 30.3R, Resistor_SMD:R_0603_1608Metric, F.Cu at (193.7, 47.3)
- added R16: 1K, Resistor_SMD:R_0603_1608Metric, F.Cu at (199.7, 50.9)
- added R17: 360R, Resistor_SMD:R_0603_1608Metric, F.Cu at (195.3, 47.3)
- added R18: 5.24R, Resistor_SMD:R_0603_1608Metric, F.Cu at (192.1, 47.3)
- added R19: 100K, Resistor_SMD:R_0603_1608Metric, F.Cu at (190.5, 47.3)
- added R2: 10K, Resistor_SMD:R_0603_1608Metric, F.Cu at (202.9, 27.1)
- added R20: 0R, Resistor_SMD:R_2010_5025Metric, F.Cu at (203.6, 54.4)
- added R21: 100R, Resistor_SMD:R_0603_1608Metric, F.Cu at (183.4, 46.5)
- added R22: 100k, PCM_SparkFun-Resistor:R_0603_1608Metric, F.Cu at (185.4, 50.3)
- added R23: 0R, Resistor_SMD:R_2010_5025Metric, F.Cu at (199.6, 47.0)
- added R24: 2K, Resistor_SMD:R_0603_1608Metric, F.Cu at (176.7, 51.5)
- added R25: 1K, Resistor_SMD:R_0805_2012Metric, F.Cu at (175.2, 34.8)
- added R26: 10K, Resistor_SMD:R_0603_1608Metric, F.Cu at (175.4, 28.3)
- added R27: 1K, Resistor_SMD:R_0603_1608Metric, F.Cu at (175.4, 31.4)
- added R28: 1K, Resistor_SMD:R_0805_2012Metric, F.Cu at (179.0, 37.6)
- added R29: 0R, Resistor_SMD:R_0805_2012Metric, F.Cu at (183.3, 37.6)
- added R3: 10K, Resistor_SMD:R_0603_1608Metric, F.Cu at (227.5, 39.5)
- added R30: 1K, Resistor_SMD:R_0805_2012Metric, F.Cu at (179.0, 39.8)
- added R31: 0R, Resistor_SMD:R_0805_2012Metric, F.Cu at (183.2, 39.8)
- added R32: 1K, Resistor_SMD:R_0805_2012Metric, F.Cu at (179.0, 42.2)
- added R33: 0R, Resistor_SMD:R_0805_2012Metric, F.Cu at (183.2, 42.2)
- added R34: 30.3R, Resistor_SMD:R_0603_1608Metric, F.Cu at (193.6, 66.0)
- added R35: 1K, Resistor_SMD:R_0603_1608Metric, F.Cu at (199.6, 69.6)
- added R36: 360R, Resistor_SMD:R_0603_1608Metric, F.Cu at (195.2, 66.0)
- added R37: 5.24R, Resistor_SMD:R_0603_1608Metric, F.Cu at (192.0, 66.0)
- added R38: 100K, Resistor_SMD:R_0603_1608Metric, F.Cu at (190.4, 66.0)
- added R39: 0R, Resistor_SMD:R_2010_5025Metric, F.Cu at (203.5, 73.1)
- added R4: 4.7K, Resistor_SMD:R_0603_1608Metric, F.Cu at (211.1, 44.3)
- added R40: 100R, Resistor_SMD:R_0603_1608Metric, F.Cu at (183.3, 65.2)
- added R41: 100k, PCM_SparkFun-Resistor:R_0603_1608Metric, F.Cu at (185.3, 69.0)
- added R42: 0R, Resistor_SMD:R_2010_5025Metric, F.Cu at (199.5, 65.6)
- added R43: 2K, Resistor_SMD:R_0603_1608Metric, F.Cu at (176.6, 70.2)
- added R44: 330R, Resistor_SMD:R_0603_1608Metric, F.Cu at (227.3, 25.5)
- added R5: 4.7K, Resistor_SMD:R_0603_1608Metric, F.Cu at (212.6, 44.3)
- added R6: 4.7K, Resistor_SMD:R_0603_1608Metric, F.Cu at (214.1, 44.3)
- added R7: 330R, Resistor_SMD:R_0603_1608Metric, F.Cu at (221.6, 43.3)
- added R8: 100K, Resistor_SMD:R_0603_1608Metric, F.Cu at (245.2, 42.4)
- added R9: 100K, Resistor_SMD:R_0603_1608Metric, F.Cu at (251.2, 39.2)
- added SW1: SW_Push, Button_Switch_SMD:SW_Push_1P1T_NO_CK_KMR2, F.Cu at (233.9, 26.9)
- added SW2: SW_Push, Button_Switch_SMD:SW_Push_1P1T_NO_CK_KMR2, F.Cu at (233.9, 33.4)
- added SW3: SW_Push, Button_Switch_SMD:SW_Push_1P1T_NO_CK_KMR2, F.Cu at (233.9, 39.8)
- added TH1: NCP18XH103, Resistor_SMD:R_0603_1608Metric, B.Cu at (126.2, 58.8)
- added TH2: NCP18XH103, Resistor_SMD:R_0603_1608Metric, B.Cu at (107.8, 59.6)
- added U1: ESP32-S3-WROOM-1, RF_Module:ESP32-S3-WROOM-1, F.Cu at (215.9, 28.2)
- added U2: AP2112K-3.3, Package_TO_SOT_SMD:SOT-23-5, F.Cu at (245.5, 38.8)
- added U3: SY6970QCC, BMS:QFN-24_L4.0-W4.0-P0.50-TL-EP2.7, F.Cu at (193.0, 52.0)
- added U4: DW01A, Package_TO_SOT_SMD:SOT-23-6, F.Cu at (179.2, 51.0)
- added U5: USBLC6-2SC6, Package_TO_SOT_SMD:SOT-23-6, F.Cu at (184.6, 29.7)
- added U6: CH224K, BMS:ESSOP-10_L4.9-W3.9-P1.0-LS6.0-TL-EP, F.Cu at (179.8, 29.7)
- added U7: SY6970QCC, BMS:QFN-24_L4.0-W4.0-P0.50-TL-EP2.7, F.Cu at (192.9, 70.7)
- added U8: DW01A, Package_TO_SOT_SMD:SOT-23-6, F.Cu at (179.1, 69.7)
Routing:
- net VBUS: track 0.00 -> 169.2 mm, vias 0 -> 4
- net /CH1_V: track 0.00 -> 163.6 mm, vias 0 -> 2
- net GND: track 0.00 -> 124.7 mm, vias 0 -> 32
- net /CELL2_N: track 0.00 -> 101.6 mm, vias 0 -> 2
- net /CELL1_N: track 0.00 -> 95.5 mm
- net Net-(U7-NTC): track 0.00 -> 92.1 mm, vias 0 -> 1
- net /CELL2_P: track 0.00 -> 91.8 mm, vias 0 -> 2
- net Net-(U3-NTC): track 0.00 -> 80.1 mm, vias 0 -> 1
- net /CELL1_P: track 0.00 -> 66.4 mm
- net /CELL1_V: track 0.00 -> 50.0 mm
- net /ESP_PWR: track 0.00 -> 49.7 mm, vias 0 -> 2
- net /CH2_V: track 0.00 -> 41.2 mm
- net /WAKE: track 0.00 -> 40.6 mm
- net /SCL2: track 0.00 -> 38.9 mm, vias 0 -> 2
- net /ESP_EN: track 0.00 -> 37.9 mm, vias 0 -> 2
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- added copper zone on In2.Cu, net +3V3
- added copper zone on F.Cu, net /CELL1_N
- added copper zone on F.Cu, net /CELL1_P
- added copper zone on F.Cu, net /CELL2_N
- added copper zone on F.Cu, net /CELL2_P
- added copper zone on F.Cu, net /charge_chanel_1/CELL_P_PROT
- added copper zone on F.Cu, net /charge_chanel_2/CELL_P_PROT
- added copper zone on F.Cu, net GND
- added copper zone on In1.Cu, net GND
- added copper zone on F.Cu, net Net-(C16-Pad1)
- added copper zone on F.Cu, net Net-(C17-Pad1)
- added copper zone on F.Cu, net Net-(C7-Pad1)
- added copper zone on F.Cu, net Net-(C8-Pad1)
- added copper zone on F.Cu, net VBUS
Other:
- board outline added: 198 x 90 mm
- copper layers 2 -> 4
- board text added: "+ - + -"
- board text added: "- +"
- board text added: "0"
- board text added: "1"
- board text added: "BATT 1"
- board text added: "BATT 2"
- board text added: "BOOT"
- board text added: "BY DASHIELL RUSSELL"
- board text added: "CFG1"
- board text added: "CFG2"
- board text added: "CFG3"
- board text added: "EN"
- board text added: "FEATH"
- board text added: "J2"
- board text added: "SRAD"
- board text added: "UNSW ROCKETRY 2026 AURC NOSECONE BMS"
- board text added: "WAKE"
