File: board4_nosecone/board4_nosecone.kicad_pcb (KiCad board)
At the start: 4 copper layers, 198 x 90 mm, 101 parts, among them J1 Screw_Terminal_01x04, J2 Screw_Terminal_01x02, J3 Screw_Terminal_01x04, J4 POWER_OFF_HEADER, J5 USB_C_Receptacle_USB2.0_16P, Q1 2N7002, Q2 DMG2305UX, Q3 SI4920DY, Q4 DMG2305UX, Q5 SI4920DY, SW1 SW_Push, SW2 SW_Push, SW3 SW_Push, U1 ESP32-S3-WROOM-1, U2 AP2112K-3.3, U3 SY6970QCC, U4 DW01A, U5 USBLC6-2SC6, U6 CH224K, U7 SY6970QCC, U8 DW01A

Commit message: board4_nosecone: routing progress (+70 segments, +31 vias)
Co-Authored-By: Claude Fable 5 <noreply@anthropic.com>
Routing:
- net /CELL2_V: track 0.00 -> 15.4 mm
