File: board4_nosecone/board4_nosecone.kicad_sch (KiCad schematic)
At the start: 0 parts

Commit message: board4_nosecone: complete schematic (ESP, cells, CFG 9V, dual holder)
- ESP32-S3 block wired: dual I2C buses (no mux), diode-OR gate, USB
  programming, RGB chain, WAKE/BOOT/RESET buttons
- CH224K strapped to 9V (CFG1/2/3 all to GND)
- BH-18650-B6AA007 dual 18650 holder: symbol added to BMS lib (5-pin,
  C1+/C1-/C2+/C2-/hidden mechanical), footprint relocated to BMS.pretty
  and renamed from misfiled UNSW_ROCKETRY_LIBRARY:BMSBH-18650-B6AA007
- BT1 placed, wired to CELL1/CELL2 nets

docs/board1_fixes_todo.md: main-board bugs found during the copy -
CFG2/CFG3 floating (PD not deterministically 12V), heartbeat LED
missing series resistor.

Known WIP: heartbeat LED (D1) on board4 still needs series resistor;
dangling wire stubs to clean; PD_GOOD LED (PG) unconnected; pull-pin
isolation break TBD. Verify in GUI ERC before layout.
Parts:
- added BT1: BH-18650-B6AA007, BMS:BH-18650-B6AA007, symbol BMS:BH-18650-B6AA007
- added C1: 1uF, Capacitor_SMD:C_0603_1608Metric, symbol Device:C
- added C2: 10uF, Capacitor_SMD:C_0805_2012Metric, symbol Device:C
- added C3: 100nF, Capacitor_SMD:C_0805_2012Metric, symbol Device:C
- added C4, C5: 1uF, Capacitor_SMD:C_0805_2012Metric, symbol Device:C
- added D1: LED, LED_SMD:LED_0603_1608Metric, symbol Device:LED
- added D2: MMBD4448HCQW, Package_TO_SOT_SMD:SOT-353_SC-70-5, symbol Diode:MMBD4448HCQW
- added J1, J3: Screw_Terminal_01x04, TerminalBlock_Phoenix:TerminalBlock_Phoenix_PT-1,5-4-3.5-H_1x04_P3.50mm_Horizontal, symbol Connector:Screw_Terminal_01x04
- added J2: Screw_Terminal_01x02, TerminalBlock_Phoenix:TerminalBlock_Phoenix_PT-1,5-2-3.5-H_1x02_P3.50mm_Horizontal, symbol Connector:Screw_Terminal_01x02
- added J4: POWER_OFF_HEADER, Connector_PinHeader_2.54mm:PinHeader_1x02_P2.54mm_Horizontal, symbol Connector:Conn_01x02_Pin
- added Q1: 2N7002, Package_TO_SOT_SMD:SOT-23, symbol Transistor_FET:2N7002
- added R1, R4, R5, R6: 4.7K, Resistor_SMD:R_0603_1608Metric, symbol Device:R
- added R10, R11, R2, R3: 10K, Resistor_SMD:R_0603_1608Metric, symbol Device:R
- added R12, R14, R8, R9: 100K, Resistor_SMD:R_0603_1608Metric, symbol Device:R
- added R13: 33K, Resistor_SMD:R_0603_1608Metric, symbol Device:R
- added R44, R7: 330R, Resistor_SMD:R_0603_1608Metric, symbol Device:R
- added SW1, SW2, SW3: SW_Push, Button_Switch_SMD:SW_Push_1P1T_NO_CK_KMR2, symbol Switch:SW_Push
- added U1: ESP32-S3-WROOM-1, RF_Module:ESP32-S3-WROOM-1, symbol RF_Module:ESP32-S3-WROOM-1
- added U2: AP2112K-3.3, Package_TO_SOT_SMD:SOT-23-5, symbol Regulator_Linear:AP2112K-3.3
Connections:
- new net: D2.3 (A), R10.1
- new net: D2.1 (A), R9.2
- new net: D2.5 (A), R12.2, R13.2
- new net: J4.2 (Pin_2), Q1.1 (G), R8.2
- new net: R7.2, U1.25 (IO48)
- new net: D1.2 (A), R44.1
- new net: D2.4 (A), R11.1
- new net +3V3: C2.1, C3.1, C5.1, R1.2, R2.2, R3.2, R4.2, R5.2, R6.2, U1.2 (3V3), U2.5 (VOUT)
- new net 3V3_EN: D2.2 (K), D2.2 (K), D2.2 (K), D2.2 (K), Q1.3 (D), R14.2, U2.3 (EN)
- new net BOOT: R3.1, SW3.1, U1.27 (IO0)
- new net CELL1_N: BT1.2 (C1-)
- new net CELL1_P: BT1.1 (C1+)
- new net CELL1_V: J1.3 (Pin_3), J2.1 (Pin_1)
- new net CELL2_N: BT1.4 (C2-)
- new net CELL2_P: BT1.3 (C2+)
- new net CELL2_V: J1.4 (Pin_4), J3.1 (Pin_1), J3.3 (Pin_3)
- new net CH1_V: C4.1, J1.2 (Pin_2), J4.1 (Pin_1), R9.1, SW1.1, U2.1 (VIN)
- new net CH2_V: J1.1 (Pin_1)
- new net ESP_EN: C1.2, R2.1, SW2.1, U1.3 (EN)
- new net ESP_PWR: R10.2, U1.10 (IO17)
- new net GND: C1.1, C2.2, C3.2, C4.2, C5.2, D1.1 (K), J2.2 (Pin_2), J3.2 (Pin_2), J3.4 (Pin_4), Q1.2 (S), R13.1, R14.1, R8.1, SW2.2, SW3.2, U1.1 (GND), U1.40 (GND), U1.41 (GND), U2.2 (GND)
- new net Heartbeat LED: R44.2, U1.38 (IO2)
- new net RGB_DATA: R7.1
- new net SCL1: R4.1, U1.17 (IO9)
- new net SCL2: R6.1, U1.19 (IO11)
- new net SDA1: R1.1, U1.12 (IO8)
- new net SDA2: R5.1, U1.18 (IO10)
- new net USB_N: U1.13 (USB_D-)
- new net USB_P: U1.14 (USB_D+)
- new net VBUS: R12.1
- new net WAKE: R11.2, SW1.2
- no-connect marks 0 -> 27
Other:
- added sheet USB_IN (USB_IN.kicad_sch)
- added sheet charge_chanel_1 (charge_chanel.kicad_sch)
- added sheet charge_chanel_2 (charge_chanel.kicad_sch)
- note added: "3V3 ENABLE"
- note added: "3V3 POWER SUPLY"
- note added: "3V3 Power"
- note added: "4 On conditions for 3V3"
- note added: "BATT"
- note added: "BOOT"
- note added: "BUTTONS"
- note added: "CHARGE CHANEL"
- note added: "CONNECTORS"
- note added: "ENABLE"
- note added: "ESP32-S3 For oprating LED'S & Streaming data and monitoring charging circuitry"
- note added: "ESP32-S3-WROOM"
- note added: "EXPERIMENTAL PAYLOADS"
- note added: "PRIMARY FC"
- note added: "PULL PIN"
- note added: "WAKE"
