File: board4_nosecone/charge_chanel.kicad_sch (KiCad schematic)
At the start: 26 parts, among them Q1 DMG2305UX, Q2 SI4920DY, U6 SY6970QCC, U7 DW01A

Commit message: board4_nosecone: complete schematic (ESP, cells, CFG 9V, dual holder)
- ESP32-S3 block wired: dual I2C buses (no mux), diode-OR gate, USB
  programming, RGB chain, WAKE/BOOT/RESET buttons
- CH224K strapped to 9V (CFG1/2/3 all to GND)
- BH-18650-B6AA007 dual 18650 holder: symbol added to BMS lib (5-pin,
  C1+/C1-/C2+/C2-/hidden mechanical), footprint relocated to BMS.pretty
  and renamed from misfiled UNSW_ROCKETRY_LIBRARY:BMSBH-18650-B6AA007
- BT1 placed, wired to CELL1/CELL2 nets

docs/board1_fixes_todo.md: main-board bugs found during the copy -
CFG2/CFG3 floating (PD not deterministically 12V), heartbeat LED
missing series resistor.

Known WIP: heartbeat LED (D1) on board4 still needs series resistor;
dangling wire stubs to clean; PD_GOOD LED (PG) unconnected; pull-pin
isolation break TBD. Verify in GUI ERC before layout.
Parts:
- renumbered C15 to C10, C16 to C11, C11 to C12, C10 to C6, C12 to C7, C13 to C8, C14 to C9, Q1 to Q2, Q2 to Q3, U6 to U3, U7 to U4
